File: cringenode.kicad_pcb (KiCad board)
At the start: 2 copper layers, 100 x 35 mm, 142 parts, among them J1 INA_STATE, J10 PROG_HEADER, J11 PWR_OUT_3, J13 OLED, J2 PWR_IN, J3 PWR_OUT_1, J4 PROTO, J5 PROTO, J6 PROTO, J7 PROTO, J8 USB_C_Receptacle_USB2.0, J9 PWR_OUT_2, Q1 MMBT2222A, Q10 MMBT2222A, Q11 WST03P06, Q12 S9015, Q13 MMBT2222A, Q14 MMBT2222A, Q15 MMBT2222A, Q16 MMBT2222A, Q17 WST03P06, Q18 S9015, Q19 MMBT2222A, Q2 WST03P06, Q20 AO3400A, Q21 AO3400A, Q22 S9015, Q23 AO3400A, Q3 WST03P06, Q4 S9015, Q5 MMBT2222A, Q6 MMBT2222A, Q7 WST03P06, Q8 S9015, Q9 MMBT2222A, SW1 RST, SW2 BOOT/B1, SW3 B2, U1 XL1509, U2 INA3221, U3 ESP32-C3-WROOM-02, U5 PAM8302AAD

Commit message: finish this unholy abomination
Parts:
- removed the C11 at (275.1, 89.9)
- removed the C6 at (270.3, 94.1)
- removed the C7 at (280.7, 82.4)
- removed the D4 at (80.0, 87.0)
- removed J13: OLED, Connector_PinSocket_2.54mm:PinSocket_1x04_P2.54mm_Vertical
- removed the J4 at (130.5, 85.8)
- removed the Q10 at (237.2, 118.5)
- removed Q11: WST03P06, Package_TO_SOT_SMD:SOT-23
- removed the Q5 at (268.5, 88.8)
- removed the Q7 at (220.0, 129.4)
- removed the Q8 at (273.1, 82.2)
- removed the Q9 at (251.5, 103.6)
- removed the R12 at (264.5, 96.7)
- removed the R15 at (252.3, 92.2)
- removed the R16 at (231.3, 131.1)
- removed the R17 at (264.5, 94.7)
- removed the R21 at (214.5, 128.9)
- removed the R22 at (239.1, 101.9)
- removed the R23 at (246.4, 94.6)
- removed the R26 at (214.5, 125.6)
- removed R30: 15k, Resistor_SMD:R_0402_1005Metric
- removed the R31 at (249.2, 108.9)
- removed the R32 at (241.4, 105.2)
- removed the R33 at (240.9, 118.3)
- removed the R35 at (205.8, 136.9)
- removed R60: 10k, Resistor_SMD:R_0402_1005Metric
- removed the R8 at (252.7, 110.9)
- added C12: 10u, Capacitor_SMD:C_0603_1608Metric, B.Cu at (149.2, 114.2)
- added C13: 100n, Capacitor_SMD:C_0402_1005Metric, B.Cu at (149.3, 112.5)
- added C21: 100n, Capacitor_SMD:C_0402_1005Metric, B.Cu at (90.2, 79.6)
- added C22: DNP, Capacitor_SMD:C_0402_1005Metric, B.Cu at (148.3, 94.2)
- added C23: DNP, Capacitor_SMD:C_0402_1005Metric, B.Cu at (148.3, 80.8)
- added C24: DNP, Capacitor_SMD:C_0402_1005Metric, B.Cu at (148.2, 108.4)
- added D5: LED_0603, LED_SMD:LED_0603_1608Metric_Pad1.05x0.95mm_HandSolder, F.Cu at (139.1, 71.2)
- added D8: LED_0603, LED_SMD:LED_0603_1608Metric_Pad1.05x0.95mm_HandSolder, F.Cu at (81.6, 90.2)
- added J12: TERM_BLOCK, Critbit_lib:DG235-5.0, F.Cu at (165.0, 79.0)
- added J8: INA_STA, Connector_PinHeader_2.54mm:PinHeader_2x02_P2.54mm_Vertical, F.Cu at (159.5, 110.5)
- added JP2: SolderJumper_3_Open, Jumper:SolderJumper-3_P2.0mm_Open_TrianglePad1.0x1.5mm_NumberLabels, B.Cu at (89.2, 105.5)
- added JP3: SolderJumper_3_Open, Jumper:SolderJumper-3_P2.0mm_Open_TrianglePad1.0x1.5mm_NumberLabels, B.Cu at (92.5, 105.5)
- added Q14: S9015, Package_TO_SOT_SMD:SOT-23, B.Cu at (143.2, 87.3)
- added Q15: MMBT2222A, Package_TO_SOT_SMD:SOT-23, B.Cu at (143.2, 91.2)
- added Q20: MMBT2222A, Package_TO_SOT_SMD:SOT-23, B.Cu at (146.8, 105.5)
- added Q21: WST03P06, Package_TO_SOT_SMD:SOT-23, B.Cu at (146.8, 101.5)
- added Q23: MMBT2222A, Package_TO_SOT_SMD:SOT-23, B.Cu at (143.2, 105.5)
- added R20: 10k, Resistor_SMD:R_0402_1005Metric, B.Cu at (112.1, 105.1)
- added R37: 10k, Resistor_SMD:R_0402_1005Metric, B.Cu at (81.6, 90.0)
- added R40: 10k, Resistor_SMD:R_0402_1005Metric, B.Cu at (146.4, 94.2)
- added R41: 0R/1206, Resistor_SMD:R_1206_3216Metric_Pad1.30x1.75mm_HandSolder, B.Cu at (144.0, 84.0)
- added R47: 10k, Resistor_SMD:R_0402_1005Metric, B.Cu at (144.4, 80.8)
- added R48: 470, Resistor_SMD:R_0402_1005Metric, B.Cu at (142.4, 80.8)
- added R49: 15k, Resistor_SMD:R_0402_1005Metric, B.Cu at (148.5, 103.6)
- added R50: 10k, Resistor_SMD:R_0402_1005Metric, B.Cu at (146.3, 108.4)
- added R52: 10k, Resistor_SMD:R_0402_1005Metric, B.Cu at (144.3, 108.4)
- added R53: 470, Resistor_SMD:R_0402_1005Metric, B.Cu at (142.3, 108.4)
- added SW4: B3, Button_Switch_SMD:SW_SPST_FSMSM, F.Cu at (94.0, 108.5)
- added TP1: INA_PAD, TestPoint:TestPoint_Pad_D2.5mm, F.Cu at (152.0, 85.2)
- added TP2: GND_PAD, TestPoint:TestPoint_Pad_D2.5mm, F.Cu at (146.7, 73.1)
- added TP5: INA_PAD, TestPoint:TestPoint_Pad_D2.5mm, F.Cu at (152.0, 80.2)
- added TP6: INA_PAD, TestPoint:TestPoint_Pad_D2.5mm, F.Cu at (152.0, 98.0)
- added TP9: INA_PAD, TestPoint:TestPoint_Pad_D2.5mm, F.Cu at (152.0, 103.0)
- C1: renamed from C2; footprint Capacitor_SMD:C_0603_1608Metric -> Capacitor_SMD:C_0402_1005Metric; moved to B.Cu
- C10: renamed from C8; moved to B.Cu
- C11: renamed from C9; moved to B.Cu
- C14: renamed from C12; moved to B.Cu
- C15: renamed from C13; moved to B.Cu
- C16: renamed from C18; moved to B.Cu
- C17: renamed from C14; moved to B.Cu
- C18: renamed from C15; moved to B.Cu
- C19: renamed from C16; moved to B.Cu
- C20: renamed from C17; moved to B.Cu
- C7: renamed from C4; moved to B.Cu
- C8: renamed from C5; footprint Capacitor_SMD:C_0603_1608Metric -> Capacitor_SMD:C_0402_1005Metric; moved to B.Cu
- C9: renamed from C1; moved to B.Cu
- D4: renamed from D5; footprint LED_THT:LED_D3.0mm_IRBlack -> LED_SMD:LED_0603_1608Metric_Pad1.05x0.95mm_HandSolder
- D6, D7: footprint LED_THT:LED_D3.0mm_IRBlack -> LED_SMD:LED_0603_1608Metric_Pad1.05x0.95mm_HandSolder
- J1: value INA_STATE -> IN+; footprint Connector_PinHeader_2.54mm:PinHeader_1x04_P2.54mm_Vertical -> Critbit_lib:DG235-5.0
- J10: value PROG_HEADER -> TERM_BLOCK; footprint Connector_PinHeader_2.54mm:PinHeader_1x08_P2.54mm_Vertical -> Critbit_lib:DG235-5.0
- J11: value PWR_OUT_3 -> TERM_BLOCK; footprint TerminalBlock_WAGO:TerminalBlock_WAGO_236-402_1x02_P5.00mm_45Degree -> Critbit_lib:DG235-5.0
- J2: value PWR_IN -> IN-; footprint TerminalBlock_WAGO:TerminalBlock_WAGO_236-402_1x02_P5.00mm_45Degree -> Critbit_lib:DG235-5.0
- J3: value PWR_OUT_1 -> Proto_matrix_14x9+7; footprint TerminalBlock_WAGO:TerminalBlock_WAGO_236-402_1x02_P5.00mm_45Degree -> Critbit_lib:Proto_matrix_14x9+7
- J5: value PROTO -> Lichtenprog_conn; footprint Connector_PinSocket_2.54mm:PinSocket_2x10_P2.54mm_Vertical -> Critbit_lib:Lichtenprog
- J6, J7: value PROTO -> TERM_BLOCK; footprint Connector_PinSocket_2.54mm:PinSocket_2x10_P2.54mm_Vertical -> Critbit_lib:DG235-5.0
- J9: value PWR_OUT_2 -> TERM_BLOCK; footprint TerminalBlock_WAGO:TerminalBlock_WAGO_236-402_1x02_P5.00mm_45Degree -> Critbit_lib:DG235-5.0
- JP6: renamed from JP4; moved to B.Cu
- L1: value L -> 47uH/2A; footprint Inductor_SMD:L_2512_6332Metric -> Inductor_SMD:L_Abracon_ASPI-0630LR
- Q1: footprint Buzzer_Beeper:Buzzer_TDK_PS1240P02BT_D12.2mm_H6.5mm -> Package_TO_SOT_SMD:SOT-23; moved to B.Cu
- Q10: renamed from Q15; moved to B.Cu
- Q12: value S9015 -> MMBT2222A; moved to B.Cu
- Q13: value MMBT2222A -> WST03P06; moved to B.Cu
- Q16, Q17, Q18, Q19, Q6, R45, R7, RV1: moved to B.Cu
- Q4: renamed from Q20; moved to B.Cu
- Q5: renamed from Q4; moved to B.Cu
- Q7: renamed from Q21; moved to B.Cu
- Q8: renamed from Q23; moved to B.Cu
- Q9: renamed from Q14; moved to B.Cu
- R10: renamed from R13; moved to B.Cu
- R11: renamed from R49; moved to B.Cu
- R12: renamed from R19; value 50mR/1206 -> 0R/1206
- R14: renamed from R59; moved to B.Cu
- R15: renamed from R24; moved to B.Cu
- R16: renamed from R27; moved to B.Cu
- R17: renamed from R28; moved to B.Cu
- R18: renamed from R36; footprint Resistor_SMD:R_0603_1608Metric_Pad0.98x0.95mm_HandSolder -> Resistor_SMD:R_0402_1005Metric
- R19: renamed from R37; footprint Resistor_SMD:R_0603_1608Metric_Pad0.98x0.95mm_HandSolder -> Resistor_SMD:R_0402_1005Metric
- R21: renamed from R40; moved to B.Cu
- R22: renamed from R41; moved to B.Cu
- R23: renamed from R2; moved to B.Cu
- R24: renamed from R3; moved to B.Cu
- R25: renamed from R4; moved to B.Cu
- R26: renamed from R5; moved to B.Cu
- R27: renamed from R25; moved to B.Cu
- R28: renamed from R38; moved to B.Cu
- R29: value 470 -> DNP; moved to B.Cu
- R3: renamed from R6; moved to B.Cu
- R31: renamed from R50; moved to B.Cu
- R32: renamed from R52; value 470 -> DNP; moved to B.Cu
- R33: renamed from R54; moved to B.Cu
- R34: value 470 -> 10k; moved to B.Cu
- R35: renamed from R56; moved to B.Cu
- R36: renamed from R57; moved to B.Cu
- R39, R44: value 0R/1206 -> 15k; footprint Resistor_SMD:R_1206_3216Metric_Pad1.30x1.75mm_HandSolder -> Resistor_SMD:R_0402_1005Metric; moved to B.Cu
- R4: renamed from R1; moved to B.Cu
- R42: value 15k -> 10k; moved to B.Cu
- R43: value 10k -> 470; moved to B.Cu
- R46, R51: value 470 -> 0R/1206; footprint Resistor_SMD:R_0402_1005Metric -> Resistor_SMD:R_1206_3216Metric_Pad1.30x1.75mm_HandSolder; moved to B.Cu
- R5: renamed from R10; moved to B.Cu
- R6: renamed from R47; moved to B.Cu
- R8: renamed from R14; moved to B.Cu
- R9: renamed from R11; moved to B.Cu
- SW1, SW2, SW3: footprint Button_Switch_THT:SW_PUSH_6mm_H4.3mm -> Button_Switch_SMD:SW_SPST_FSMSM
- TP10: renamed from TP5; value TestPoint -> CON_PAD; footprint Connector_PinSocket_2.54mm:PinSocket_1x01_P2.54mm_Vertical -> MountingHole:MountingHole_2.7mm_M2.5_DIN965_Pad
- TP11: renamed from TP6; value TestPoint -> CON_PAD; footprint Connector_PinSocket_2.54mm:PinSocket_1x01_P2.54mm_Vertical -> MountingHole:MountingHole_2.7mm_M2.5_DIN965_Pad
- TP3: renamed from TP1; value TestPoint -> CON_PAD; footprint Connector_PinSocket_2.54mm:PinSocket_1x01_P2.54mm_Vertical -> MountingHole:MountingHole_2.7mm_M2.5_DIN965_Pad
- TP4: renamed from TP2; value TestPoint -> CON_PAD; footprint Connector_PinSocket_2.54mm:PinSocket_1x01_P2.54mm_Vertical -> MountingHole:MountingHole_2.7mm_M2.5_DIN965_Pad
- TP7: renamed from TP3; value TestPoint -> CON_PAD; footprint Connector_PinSocket_2.54mm:PinSocket_1x01_P2.54mm_Vertical -> MountingHole:MountingHole_2.7mm_M2.5_DIN965_Pad
- TP8: renamed from TP4; value TestPoint -> CON_PAD; footprint Connector_PinSocket_2.54mm:PinSocket_1x01_P2.54mm_Vertical -> MountingHole:MountingHole_2.7mm_M2.5_DIN965_Pad
- U4: renamed from U5; moved to B.Cu
- moved Q5 194.0 mm to (84.2, 91.6), turned to 180 degrees
- moved R16 184.8 mm to (87.4, 84.8), turned to -90 degrees
- moved Q6 184.0 mm to (89.6, 87.0), turned to -90 degrees
- moved R8 182.3 mm to (104.5, 100.4), turned to 90 degrees
- moved Q1 180.5 mm to (88.2, 91.6), turned to 180 degrees
- moved C16 176.1 mm to (99.0, 89.5)
- moved R17 175.5 mm to (87.4, 79.7), turned to 90 degrees
- moved C7 172.1 mm to (97.2, 102.2), turned to -90 degrees
- moved R4 171.7 mm to (89.0, 89.4), turned to 180 degrees
- moved R7 169.8 mm to (86.0, 89.3), turned to 180 degrees
- moved C20 169.4 mm to (104.8, 107.5), turned to -90 degrees
- moved C9 164.1 mm to (83.2, 89.3), turned to 180 degrees
- moved R9 158.1 mm to (87.4, 86.8), turned to -90 degrees
- moved R10 158.0 mm to (89.5, 84.4)
- moved C14 152.2 mm to (111.9, 77.1)
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- renumbered C3 to C2, C19 to C3, C20 to C4, C21 to C5, C22 to C6, J8 to J4, JP2 to JP4, JP3 to JP5, R18 to R1, R9 to R13, R20 to R2, U3 to U2, U2 to U3
Connections:
- net Net-(C2-Pad1) renamed /DCDC_L
- net Net-(J11-Pad1) renamed /TERM5
- net Net-(J8-PadA6) renamed /USBDP
- net Net-(J8-PadA7) renamed /USBDM
- net Net-(J9-Pad1) renamed /TERM3
- net Net-(L1-Pad1) renamed /DCDC_OUT
- C15 pad 1: /BOOT_BUT1 -> /IO9/BOOT_BUT1
- C16 pad 1: /BUT2 -> /IO8/BUT2
- C17 pad 1: Net-(C14-Pad1) -> /3V3_SPK
- C18 pad 2: Net-(C14-Pad1) -> /3V3_SPK
- C20 pad 1: /SPK_PWM -> GND
- C9 pad 1: /OUT3_CTRL -> /IO7/GATE_IN
- D1 pad 2: /PWRIN_LED -> /V_IN
- D4 pad 2: /PWRIN_LED -> /V_IN
- D7 pad 2: /STA_LED -> /IO7/GATE_IN
- H3 pad 1: GND -> /HACHET_FILL_NC
- H4 pad 1: GND -> /HACHET_FILL_NC
- J1 pad 1: Net-(J1-Pad1) -> /V_IN
- J10 pad 1: Net-(J10-Pad1) -> /TERM4
- J2 pad 1: /PWRIN_LED -> /V_IN_GND
- J5 pad 1: +3.3V -> Net-(J5-Pad1)
- J5 pad 2: unconnected-(J5-Pad2) -> /RTS
- J5 pad 3: unconnected-(J5-Pad3) -> /DTR
- J5 pad 4: unconnected-(J5-Pad4) -> /TARG_TX
- J5 pad 5: unconnected-(J5-Pad5) -> /TARG_RX
- J5 pad 6: unconnected-(J5-Pad6) -> GND
- J5 pad 7: unconnected-(J5-Pad7) -> GND
- J5 pad 8: unconnected-(J5-Pad8) -> Net-(J5-Pad8)
- J6 pad 1: VBUS -> /TERM1
- J7 pad 1: +VDC -> /TERM2
- JP1 pad 1: /PWRIN_LED -> /V_IN
- JP4 pad 1: Net-(J10-Pad1) -> Net-(J5-Pad1)
- JP5 pad 1: Net-(J10-Pad8) -> Net-(J5-Pad8)
- JP6 pad 1: Net-(C14-Pad1) -> /3V3_SPK
- Q10 pad 3: /IO9 -> /IO9/BOOT_BUT1
- Q12 pad 1: Net-(Q10-Pad1) (its old number) -> Net-(Q12-Pad1)
- Q12 pad 2: Net-(Q10-Pad2) -> Net-(Q12-Pad2)
- Q12 pad 3: GND -> +VDC
- Q13 pad 1: Net-(C7-Pad2) -> Net-(Q12-Pad2)
- Q13 pad 2: Net-(Q13-Pad2) -> /High side load switch1/PMOS_PWRPAD
- Q13 pad 3: Net-(Q10-Pad1) (its old number) -> +VDC
- Q17 pad 2: Net-(Q17-Pad2) -> /High side load switch/PMOS_PWRPAD
- Q19 pad 1: Net-(C11-Pad2) -> Net-(C23-Pad2)
- Q2 pad 2: Net-(Q2-Pad2) -> +VDC
- Q2 pad 3: /PWRIN_LED -> Net-(Q2-Pad3)
- Q22 pad 2: +3.3V -> Net-(Q20-Pad2)
- Q22 pad 3: Net-(D4-Pad2) -> GND
- Q3 pad 2: Net-(Q2-Pad2) -> +VDC
- Q3 pad 3: /PWRIN_LED -> Net-(Q2-Pad3)
- R1 pad 1: GND -> /V_IN
- R1 pad 2: Net-(J2-Pad2) -> Net-(Q2-Pad3)
- R12 pad 2: Net-(J2-Pad2) -> /V_IN_GND
- R13 pad 1: Net-(Q2-Pad2) -> GND
- R13 pad 2: +VDC -> /V_IN_GND
- R18 pad 1: /I2C_SCL -> /IO5/SCL
- R19 pad 1: /I2C_SDA -> /IO6/SDA
- R2 pad 1: GND -> /V_IN
- R2 pad 2: Net-(J2-Pad2) -> Net-(Q2-Pad3)
- R23 pad 1: Net-(J1-Pad4) -> Net-(R23-Pad1)
- R24 pad 1: Net-(J1-Pad3) -> Net-(R24-Pad1)
- R25 pad 1: Net-(J1-Pad2) -> Net-(R25-Pad1)
- R26 pad 1: Net-(J1-Pad1) -> Net-(R26-Pad1)
- R27 pad 1: /OUT1_GND -> Net-(U3-Pad12)
- R27 pad 2: GND -> Net-(U3-Pad11)
- R28 pad 1: /OUT2_GND -> Net-(U3-Pad15)
- R28 pad 2: GND -> Net-(U3-Pad14)
- R29 pad 1: /TARG_TX -> Net-(R31-Pad2)
- R29 pad 2: Net-(R29-Pad2) -> /IO10/SPK_PWM
- R31 pad 2: Net-(R50-Pad2) -> Net-(R31-Pad2)
- R32 pad 1: /SPK_PWM -> GND
- R34 pad 2: Net-(Q13-Pad2) -> Net-(D5-Pad1)
- R39 pad 1: /OUT2_SNUNTN -> Net-(Q12-Pad1)
- R39 pad 2: GND -> +VDC
- R4 pad 2: /PWRIN_LED -> /V_IN
- R42 pad 1: Net-(Q16-Pad1) -> GND
- R42 pad 2: +VDC -> Net-(C22-Pad2)
- R43 pad 1: Net-(C11-Pad2) -> GND
- R43 pad 2: /GATE_O3 -> Net-(Q15-Pad2)
- R44 pad 1: Net-(Q17-Pad2) -> Net-(Q16-Pad1)
- R44 pad 2: /OUT3_PWR -> +VDC
- R45 pad 1: GND -> Net-(C23-Pad2)
- R45 pad 2: Net-(C11-Pad2) -> /GATE_O1
- R46 pad 1: GND -> /High side load switch/PMOS_PWRPAD
- R46 pad 2: Net-(Q19-Pad2) -> /OUT1_PWR
- R51 pad 1: GND -> /High side load switch2/PMOS_PWRPAD
- R51 pad 2: Net-(D4-Pad1) (its old number) -> /OUT3_PWR
- R7 pad 2: /OUT3_CTRL -> /IO7/GATE_IN
- RV1 pad 1: Net-(C14-Pad1) -> /IO10/SPK_PWM
- RV1 pad 2: Net-(C14-Pad1) -> /IO10/SPK_PWM
- RV1 pad 3: Net-(R50-Pad2) -> Net-(R31-Pad2)
- SW2 pad 2: /BOOT_BUT1 -> /IO9/BOOT_BUT1
- SW3 pad 2: /BUT2 -> /IO8/BUT2
- TP11 pad 1: Net-(J11-Pad2) -> /TERM6
- TP3 pad 1: Net-(J3-Pad1) -> /TERM1
- TP4 pad 1: Net-(J3-Pad2) -> /TERM2
- TP8 pad 1: Net-(J9-Pad2) -> /TERM4
- U2 pad 10: /SPK_PWM -> /IO10/SPK_PWM
- U2 pad 12: Net-(R29-Pad2) -> /TARG_TX
- U2 pad 15: /IO3 -> /IO3/BUT3
- U2 pad 3: /IO4 -> /IO4/LED
- U2 pad 4: /I2C_SCL -> /IO5/SCL
- U2 pad 5: /I2C_SDA -> /IO6/SDA
- U2 pad 6: /IO7 -> /IO7/GATE_IN
- U2 pad 7: /BUT2 -> /IO8/BUT2
- U2 pad 8: /BOOT_BUT1 -> /IO9/BOOT_BUT1
- U3 pad 1: /OUT2_SNUNTN -> /VIN_SHUNTN
- U3 pad 10: Net-(J1-Pad1) -> Net-(R26-Pad1)
- U3 pad 11: /VIN_SHUNTN -> Net-(U3-Pad11)
- U3 pad 12: /VIN_SHUNTP -> Net-(U3-Pad12)
- U3 pad 13: Net-(J1-Pad4) -> Net-(R23-Pad1)
- U3 pad 14: /OUT1_SNUNTN -> Net-(U3-Pad14)
- U3 pad 15: /OUT1_SHUNTP -> Net-(U3-Pad15)
- U3 pad 2: /OUT2_SHUNTP -> /VIN_SHUNTP
- U3 pad 6: /I2C_SCL -> /IO5/SCL
- U3 pad 7: /I2C_SDA -> /IO6/SDA
- U3 pad 8: Net-(J1-Pad3) -> Net-(R24-Pad1)
- U3 pad 9: Net-(J1-Pad2) -> Net-(R25-Pad1)
- U4 pad 1: +3.3V -> /3V3_SPK
- U4 pad 6: Net-(C14-Pad1) -> /3V3_SPK
Routing:
- net GND: track 0.00 -> 266.4 mm, vias 0 -> 25
- net VBUS: track 0.00 -> 107.5 mm, vias 0 -> 4
- net +3.3V: track 0.00 -> 105.3 mm, vias 0 -> 5
- net /IO7/GATE_IN: track 0.00 -> 99.0 mm, vias 0 -> 5
- net /IO9/BOOT_BUT1: track 0.00 -> 78.4 mm, vias 0 -> 6
- net /VIN_SHUNTP: track 0.00 -> 72.8 mm, vias 0 -> 1
- net /IO5/SCL: track 0.00 -> 72.3 mm, vias 0 -> 1
- net /IO6/SDA: track 0.00 -> 71.8 mm, vias 0 -> 1
- net /VIN_SHUNTN: track 0.00 -> 70.6 mm, vias 0 -> 1
- net /IO10/SPK_PWM: track 0.00 -> 61.6 mm, vias 0 -> 1
- net /IO4/LED: track 0.00 -> 60.5 mm, vias 0 -> 2
- net /GATE_B: track 0.00 -> 54.8 mm, vias 0 -> 1
- net /IO3/BUT3: track 0.00 -> 53.1 mm, vias 0 -> 2
- net /GATE_G: track 0.00 -> 52.2 mm, vias 0 -> 2
- net /GATE_R: track 0.00 -> 51.9 mm
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- added copper zone on B.Cu, net +3.3V
- added copper zone on F.Cu, net +3.3V
- added copper zone on B.Cu, net +VDC
- added copper zone on F.Cu, net +VDC
- added copper zone on B.Cu, net /DCDC_L
- added copper zone on B.Cu, net /DCDC_OUT
- added copper zone on B.Cu, net /HACHET_FILL_NC
- added copper zone on F.Cu, net /HACHET_FILL_NC
- added copper zone on B.Cu, net /High side load switch/PMOS_PWRPAD
- added copper zone on B.Cu, net /High side load switch1/PMOS_PWRPAD
- added copper zone on B.Cu, net /High side load switch2/PMOS_PWRPAD
- added copper zone on B.Cu, net /OUT1_PWR
- added copper zone on B.Cu, net /OUT2_PWR
- added copper zone on F.Cu, net /OUTR
- added copper zone on B.Cu, net /TERM1
- added copper zone on F.Cu, net /TERM1
- added copper zone on B.Cu, net /TERM2
- added copper zone on F.Cu, net /TERM2
- added copper zone on B.Cu, net /TERM3
- added copper zone on F.Cu, net /TERM3
- added copper zone on B.Cu, net /TERM4
- added copper zone on F.Cu, net /TERM4
- added copper zone on B.Cu, net /TERM5
- added copper zone on F.Cu, net /TERM5
- added copper zone on B.Cu, net /TERM6
- added copper zone on F.Cu, net /TERM6
- added copper zone on B.Cu, net GND
- added copper zone on F.Cu, net GND
Other:
- board size 100 x 35 mm -> 121.9 x 47 mm
- board text added: "(C) critbit@vcc.earth"
- board text added: "5V"
- board text added: "B1"
- board text added: "B2"
- board text added: "B3"
- board text added: "CH1"
- board text added: "CH2"
- board text added: "CringeNode r. 1.0"
- board text added: "G1"
- board text added: "G2"
- board text added: "G3"
- board text added: "INA3221 Current meas."
- board text added: "IO10/SPK"
- board text added: "IO3/B3"
- board text added: "IO4/LED"
- board text added: "IO5/SCL"
- board text added: "IO6/SDA"
- board text added: "IO7/G_IN"
- board text added: "IO9/B1"
- board text added: "OLED"
- board text added: "RST"
- board text added: "SPKR+"
- board text added: "SPKR-"
- board text added: "STATUS"
- board text added: "VDC_ENA"
- board text added: "VIN"
- board text removed: "3v3"
- board text removed: "DTR"
- board text removed: "ESP32-C3 pins"
- board text removed: "ESP_RX"
- board text removed: "ESP_TX"
- board text removed: "G1 G2 G3 GR GG GB"
- board text removed: "HB"
- board text removed: "INA_S1"
- board text removed: "INA_S2"
- board text removed: "IO3"
- board text removed: "IO4"
- board text removed: "IO7"
- board text removed: "MOS gates:"
- board text removed: "OLED be here"
- board text removed: "PROG_3V3"
- board text removed: "PROG_5V"
- board text removed: "PWR"
- board text removed: "Prog con:"
- board text removed: "RTS"
- board text removed: "SCL/IO5"
- board text removed: "SDA/IO6"
- board text removed: "SPKR"
- board text removed: "TX"
- board text removed: "To ckeck: snapmount FPs smolest LEDs smolest tht buttons INA3221? inductors? Rsense? Mosfets???"
