File: cringenode.kicad_sch (KiCad schematic)
At the start: 22 parts, among them Q801 L8050QLT1G

Commit message: changes
Parts:
- added C? (x2): TBD, Capacitor_SMD:C_0402_1005Metric, symbol Device:C_Small
- added C? (x2): 15p, Capacitor_SMD:C_0402_1005Metric, symbol Device:C_Small
- added J?: PWR_OUT_1, symbol Connector:Screw_Terminal_01x02
- added J?: USB_C_PWRONLY, symbol Connector_Generic:Conn_01x02
- added J?: PWR_OUT_3, symbol Connector:Screw_Terminal_01x02
- added J?: PWR_IN, symbol Connector:Screw_Terminal_01x02
- added J?: Conn_01x05, symbol Connector_Generic:Conn_01x05
- added J?: PWR_OUT_2, symbol Connector:Screw_Terminal_01x02
- added L?: TBD, symbol Device:L_Small
- Y?: value 40MHz -> 40MHz_3225
Connections:
- net ESP_EN: now also U?.7 (CHIP_EN)
- net GND: now also Y?.1, Y?.3, C?.2, C?.2, C?.2, C?.2, J?.2 (Pin_2), J?.2 (Pin_2), J?.2 (Pin_2), J?.2 (Pin_2), J?.2 (Pin_2)
- net at U?.1 (LNA_IN): now also C?.1, L?.2
- net at U?.29 (XTAL_N): now also Y?.4, C?.1
- net at U?.30 (XTAL_P): now also Y?.2, C?.1
- new net +VDC: J?.1 (Pin_1), J?.1 (Pin_1)
- new net Antenna: C?.1, L?.1
- no-connect marks 1 -> 2
Other:
- moved on the sheet: C?, R?, Y?

Commit message: work rly hard on schematic
Parts:
- removed C?: 10u, Capacitor_SMD:C_0603_1608Metric, symbol Device:C_Small
- removed C? (x2): 100n, Capacitor_SMD:C_0402_1005Metric, symbol Device:C_Small
- removed FB?: 0R/1206, Inductor_SMD:L_1206_3216Metric, symbol Device:FerriteBead
- removed J?: Conn_01x05, Connector_PinHeader_2.54mm:PinHeader_1x05_P2.54mm_Vertical, symbol Connector_Generic:Conn_01x05
- removed J?: USB_C_PWRONLY, symbol Connector_Generic:Conn_01x02
- removed J?: Conn_01x05, symbol Connector_Generic:Conn_01x05
- removed J?: Conn_01x13, Connector_PinHeader_2.54mm:PinHeader_1x13_P2.54mm_Vertical, symbol Connector_Generic:Conn_01x13
- removed R? (x5): 10k, Resistor_SMD:R_0402_1005Metric, symbol Device:R
- removed R?: 499R, Resistor_SMD:R_0402_1005Metric, symbol Device:R
- added BZ?: Buzzer_DNP, symbol Device:Buzzer
- added C? (x6): 100n, Capacitor_SMD:C_0603_1608Metric, symbol Device:C_Small
- added C? (x7): 10u, Capacitor_SMD:C_0603_1608Metric, symbol Device:C_Small
- added C? (x12): 100n, Capacitor_SMD:C_0402_1005Metric, symbol Device:C_Small
- added C?: 330uF/6.3V, symbol Device:C_Polarized_Small_US
- added C? (x2): 10n, Capacitor_SMD:C_0603_1608Metric, symbol Device:C_Small
- added C? (x3): 4.7u, Capacitor_SMD:C_0402_1005Metric, symbol Device:C_Small
- added C?: 47uF/6.3V, Capacitor_SMD:C_0603_1608Metric, symbol Device:C_Small
- added D? (x3): SS54, symbol Device:D_Schottky
- added D? (x3): LED_0603, LED_SMD:LED_0603_1608Metric, symbol Device:LED
- added J?: WS2812_OUT, symbol Connector_Generic:Conn_01x03
- added J?: RGB_OUT, symbol Connector_Generic:Conn_01x04
- added J?: USB_C_Receptacle_USB2.0, Connector_USB:USB_C_Receptacle_HRO_TYPE-C-31-M-12, symbol Connector:USB_C_Receptacle_USB2.0
- added JP? (x2): PWR_FROM_USBC, symbol Jumper:SolderJumper_2_Open
- added JP?: 3V3_FROM_USBC, symbol Jumper:SolderJumper_2_Open
- added L?: 2nH, symbol Device:L_Small
- added L?: L, symbol Device:L
- added LS?: Speaker, symbol Device:Speaker
- added Q? (x3): AO3400A, Package_TO_SOT_SMD:SOT-23, symbol Transistor_FET:AO3400A
- added Q? (x5): 2N7002, Package_TO_SOT_SMD:SOT-23, symbol Transistor_FET:2N7002
- added Q? (x4): WST03P06, Package_TO_SOT_SMD:SOT-23, symbol Critbit_lib:WST03P06
- added R? (x18): 10k, Resistor_SMD:R_0402_1005Metric, symbol Device:R_Small
- added R? (x4): 100mR/1206, Resistor_SMD:R_1206_3216Metric_Pad1.30x1.75mm_HandSolder, symbol Device:R
- added R? (x4): 3k, Resistor_SMD:R_0603_1608Metric_Pad0.98x0.95mm_HandSolder, symbol Device:R_Small
- added R? (x6): 0R/1206, Resistor_SMD:R_1206_3216Metric_Pad1.30x1.75mm_HandSolder, symbol Device:R
- added R? (x8): 2R/1206, Resistor_SMD:R_1206_3216Metric_Pad1.30x1.75mm_HandSolder, symbol Device:R
- added R? (x6): 470, Resistor_SMD:R_0402_1005Metric, symbol Device:R_Small
- added R?: 910k, Resistor_SMD:R_0402_1005Metric, symbol Device:R_Small
- added R?: 0R/1206, Resistor_SMD:R_0402_1005Metric, symbol Device:R_Small
- added SW?: B2, Byotta:SW_ALPS_SKRKAEE020, symbol Switch:SW_Push
- added U?: PCA9557PW, Package_SO:TSSOP-16_4.4x5mm_P0.65mm, symbol Interface_Expansion:PCA9557PW
- added U? (x4): INA181, Package_TO_SOT_SMD:SOT-23-6, symbol Amplifier_Current:INA181
- added U?: XL1509, Package_SO:SOIC-8_3.9x4.9mm_P1.27mm, symbol Critbit_lib:XL1509
- added U?: JLC_OLED, symbol Critbit_lib:JLC_OLED
- added U?: PAM8302AAD, symbol Amplifier_Audio:PAM8302AAD
- D?: value LED -> LED_0603
- SW?: value BOOT -> RST
- SW?: value RST -> BOOT/B1
Connections:
- net IO7 is gone; now on net +3.3V: D?.2 (A)
- net +3.3V: now also U?.11 (VDD3P3_RTC), U?.17 (VDD3P3_CPU), U?.31 (VDDA), U?.32 (VDDA), C?.1, C?.1, C?.1, C?.1, C?.1, C?.1, C?.1, C?.1, C?.1, C?.1, C?.1, C?.1, C?.2, C?.2, C?.2, C?.2, D?.2 (A), JP?.2 (B), L?.1, L?.2, R?.2, R?.2, R?.2, U?. (~{RST}), U?.1 (~{SD}), U?.16 (VDD), U?.6 (V+), U?.6 (V+), U?.6 (V+), U?.6 (V+), U?.6 (VDD)
- net +VDC: now also J?.1 (Pin_1), J?.1 (Pin_1), Q?.3 (D), Q?.3 (D), Q?.3 (D), R?.2, R?.2, R?.2, R?.2; no longer J?.1 (Pin_1)
- net DTR: now also R?.1
- net ESP_EN: now also R?.1
- net GND: now also U?.33 (GND), C?.1, C?.1, C?.1, C?.1, C?.1, C?.1, C?.1, C?.1, C?.1, C?.2, C?.2, C?.2, C?.2, C?.2, C?.2, C?.2, C?.2, C?.2, C?.2, C?.2, C?.2, C?.2, C?.2, C?.2, D?.2 (A), J?.3 (Pin_3), J?.A1 (GND), J?.A12 (GND), J?.B1 (GND), J?.B12 (GND), J?.S1 (SHIELD), Q?.2 (S), Q?.2 (S), Q?.2 (S), Q?.2 (S), Q?.2 (S), Q?.2 (S), Q?.2 (S), Q?.2 (S), R?.1, R?.1, R?.1, R?.1, R?.1, R?.1, R?.1, R?.1, R?.1, R?.1, R?.1, R?.1, R?.1, R?.1, R?.1, R?.2, R?.2, R?.2, R?.2, R?.2, R?.2, R?.2, R?.2, R?.2, SW?.1, U?. (~{RST}), U?.2 (GND), U?.2 (GND), U?.2 (GND), U?.2 (GND), U?.3 (A0), U?.4 (A1), U?.4 (~{ON}/OFF), U?.5 (A2), U?.5 (GND), U?.5 (REF), U?.5 (REF), U?.5 (REF), U?.5 (REF), U?.6 (GND), U?.7 (GND), U?.7 (GND), U?.8 (GND), U?.8 (VSS); no longer J?.2 (Pin_2), J?.2 (Pin_2), J?.2 (Pin_2), J?.2 (Pin_2)
- net IO8: now also U?.14 (GPIO8), C?.1, R?.1, SW?.2
- net IO9: now also U?.15 (GPIO9/BOOT)
- net RTS: now also R?.1
- net TARG_RX: now also U?.27 (U0RXD/GPIO20)
- net TARG_TX: now also Q?.1 (G), R?.1
- net OUT1_PWR: now reaches J?.1 (Pin_1)
- net OUT1_PWR: now also R?.2
- net I2C_SCL: now reaches U?.10 (MTDI/GPIO5/ADC2_CH0)
- net I2C_SCL: now also U?. (~{RST}), U?.1 (SCL)
- net I2C_SDA: now reaches U?.12 (MTCK/GPIO6)
- net I2C_SDA: now also U?. (~{RST}), U?.2 (SDA)
- net I2C_RST: now reaches U?.13 (MTDO/GPIO7)
- net I2C_RST: now also U?. (~{RST}), U?.15 (~{RESET})
- net WS2812_CTRL: now reaches U?.16 (GPIO10)
- net WS2812_CTRL: now also J?.2 (Pin_2)
- net at U?.2 (VDD3P3): now also U?.3 (VDD3P3), C?.1, L?.2
- net at U?.25 (GPIO18/USB_D-): now also J?.A7 (D-), J?.B7 (D-)
- net at U?.26 (GPIO19/USB_D+): now also J?.A6 (D+), J?.B6 (D+)
- net at U?.28 (U0TXD/GPIO21): now also R?.2
- net ADC0: now reaches U?.4 (XTAL_32K_P/ADC1_CH0)
- net ADC0: now also U?.1
- net ADC1: now reaches U?.5 (XTAL_32K_N/ADC1_CH1)
- net ADC1: now also U?.1
- net ADC2: now reaches U?.6 (GPIO2/ADC1_CH2)
- net ADC2: now also U?.1
- net ADC3: now reaches U?.8 (GPIO3/ADC1_CH3)
- net ADC3: now also R?.1, R?.2
- net SPK_PWM: now reaches U?.9 (MTMS/GPIO4/ADC1_CH4)
- net SPK_PWM: now also R?.2
- net at D?.1 (K): now also R?.2
- net at Q801.1 (B): now also R?.2
- net OUT3_PWR: now reaches J?.1 (Pin_1)
- net OUT3_PWR: now also R?.2
- net at J?.1 (Pin_1): now also JP?.1 (A)
- net at J?.8 (Pin_8): now also JP?.1 (A)
- net OUT2_PWR: now reaches J?.1 (Pin_1)
- net OUT2_PWR: now also R?.2
- net at Q?.1 (B): now also R?.2
- new net: J?.3 (Pin_3), Q?.3 (D)
- new net: Q?.1 (G), R?.2
- new net: C?.1, C?.1, D?.1 (K), D?.1 (K), U?.1 (VIN)
- new net: Q?.1 (G), Q?.3 (D), R?.1 (x4)
- new net: J?.2 (Pin_2), R?.2, R?.2
- new net: C?.1, R?.1, U?.3 (+) (x4)
- new net: C?.2, R?.1, U?.4 (-) (x4)
- new net: C?.1, U?. (~{RST}) (x2)
- new net: C?.2, U?. (~{RST}) (x2)
- new net: D?.1 (K), R?.2 (x3)
- new net: Q?.2 (S), R?.1 (x4)
- new net: C?.2, U?.4 (IN-)
- new net: C?.1, R?.1, R?.2
- new net: R?.1, U?.5 (OUT+)
- new net: LS?.1, R?.2
- new net: C?.2, C?.2, U?. (~{RST}) (x2)
- new net: J?.4 (Pin_4), Q?.3 (D)
- new net: D?.1 (K), L?.1, U?.2 (OUT)
- new net: C?.2, R?.1, R?.2, U?.3 (FB)
- new net: Q?.3 (D), R?.1
- new net: R?.1, U?.8 (OUT-)
- new net: LS?.2, R?.2
- new net: J?.A5 (CC1), R?.1
- new net: R?.2, U?. (~{RST})
- new net: BZ?.2 (+), R?.2
- new net: C?.2, U?.3 (IN+)
- new net: J?.B5 (CC2), R?.1
- new net: J?.2 (Pin_2), Q?.3 (D)
- new net OUT1_CTRL: Q?.1 (G), R?.2, U?.12 (IO5)
- new net OUT1_GND: J?.2 (Pin_2), R?.1, R?.2
- new net OUT2_CTRL: Q?.1 (G), R?.2, U?.13 (IO6)
- new net OUT2_GND: J?.2 (Pin_2), R?.1, R?.2
- new net OUT3_CTRL: Q?.1 (G), R?.2, U?.14 (IO7)
- new net OUT3_GND: J?.2 (Pin_2), R?.1, R?.2
- new net OUTB_CTRL: Q?.1 (G), R?.2, U?.11 (IO4)
- new net OUTG_CTRL: Q?.1 (G), R?.2, U?.10 (IO3)
- new net OUTR_CTRL: Q?.1 (G), R?.2, U?.9 (IO2)
- new net PWRIN_LED: D?.2 (A), D?.2 (A), J?.1 (Pin_1), JP?.1 (A), Q?.3 (D), R?.2, R?.2
- new net STA_BUZZ: BZ?.1 (-), U?.7 (IO1)
- new net STA_LED: D?.2 (A), U?.6 (IO0)
- new net VBUS: D?.2 (A), J?.A4 (VBUS), J?.A9 (VBUS), J?.B4 (VBUS), J?.B9 (VBUS), JP?.2 (B), JP?.2 (B)
- no-connect marks 2 -> 10
Other:
- note added: "$0.20"
- note added: "1.8V@40Vin"
- note added: "CHECK PINOUT!!!!!!"
- note added: "For Hfe in range 150-300: Ibe = (3.3V - 0.7V)/R? Assume Ibe=10uA R? = 2.7/10uA = 2.7*100k = 270k for Ibe=10uA Ice range is [1.5-3]mA Assume VDC=5V, Rgs=10k Ugs = 10k*1mA = 10V"
- note added: "VIN range 5-40V"
- note added: "https://www.falstad.com/circuit/circuitjs.html?ctz=CQAgjCAMB0l3BWKsAsBOATCgbCjAOAdm0IRUjXxGwxCRQGY6BTAWjDACgxDbWtI4bIP7kQKKoMJ1xgpIJhIAagHsANgBcAhgHNmnHSFb45YPiboEoUTgCcjFsMIeCGkFNbdxOAdxdCRHmwAmz92YhA3D2NXdxsAByMgyLjw4KdBCAVff3IRCyibACUQDF5ZQQIqBgwFazEGaCY6xU4AMySIwtFYjwYmMGgkRtIDIwFxXHGxBCtssImq6cznSBy0kJ6QtYBjTuDu5MZaWjA2NHAmyAQEBnJ0BGwwSCxkOC5DDeP9y0kbey2NREExwHkyaw6rBq4icuVh0MGtBgLzsuWhMToZm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"
- note added: "https://www.falstad.com/circuit/circuitjs.html?ctz=CQAgjCAMB0l3BWKsDMCBMAOAbNymwAWBTTQzAThG3RCUJToFMBaMMAKDAHZaX1CkcHhD9BIclBDcQWWZilCYSAGoB7ADYAXAIYBzJhz2jMQhn1N05SjgCcTQsCJaWUkQlLDxIHAF5S3D0cRWgATJgAzHQBXbRZfJgA7JlsOAHcHYSE2bmwsqHTRHjzAzNKfAAci3JBSnLynR0UOLVEUWkInTM68pv5uaGxSTBQUbkx0SBJ0WhgUdjhCLF5JhEh0GTwhcKjYrUKXMzgy9wL7FnaJLskeqQ3vQpuu4qvewuDsy0aCjKE611OPgASuAaqUwBRaDMglJxChoIwlMgEBwItUSqcxH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"
- moved on the sheet: C?, D?, J?, L?, Q801, Q?, SW?, U?, Y?

Commit message: mostly finishing schematic
Parts:
- removed C? (x7): 100n, Capacitor_SMD:C_0402_1005Metric, symbol Device:C_Small
- removed C?: 10u, Capacitor_SMD:C_0603_1608Metric, symbol Device:C_Small
- removed C? (x3): 4.7u, Capacitor_SMD:C_0402_1005Metric, symbol Device:C_Small
- removed R? (x3): 100mR/1206, Resistor_SMD:R_1206_3216Metric_Pad1.30x1.75mm_HandSolder, symbol Device:R
- removed R? (x3): 3k, Resistor_SMD:R_0603_1608Metric_Pad0.98x0.95mm_HandSolder, symbol Device:R_Small
- removed R? (x4): 10k, Resistor_SMD:R_0402_1005Metric, symbol Device:R_Small
- removed R? (x2): 2R/1206, Resistor_SMD:R_1206_3216Metric_Pad1.30x1.75mm_HandSolder, symbol Device:R
- removed R?: 910k, Resistor_SMD:R_0402_1005Metric, symbol Device:R_Small
- removed U?: INA181, Package_TO_SOT_SMD:SOT-23-6, symbol Amplifier_Current:INA181
- removed U?: JLC_OLED, symbol Critbit_lib:JLC_OLED
- added C?: 100n, Capacitor_SMD:C_0402_1005Metric, symbol Device:C_Small
- added C?: 10u, Capacitor_SMD:C_0603_1608Metric, symbol Device:C_Small
- added J?: OLED, symbol Connector_Generic:Conn_01x04
- added JP?: SPK_ENA, symbol Jumper:SolderJumper_2_Open
- added Q?: WST03P06, Package_TO_SOT_SMD:SOT-23, symbol Critbit_lib:WST03P06
- added R? (x3): 10k, Resistor_SMD:R_0402_1005Metric, symbol Device:R_Small
- added R? (x4): 50mR/1206, Resistor_SMD:R_1206_3216Metric_Pad1.30x1.75mm_HandSolder, symbol Device:R
- added R? (x2): 3k, Resistor_SMD:R_0603_1608Metric_Pad0.98x0.95mm_HandSolder, symbol Device:R_Small
- added R? (x3): 5k, Resistor_SMD:R_0603_1608Metric_Pad0.98x0.95mm_HandSolder, symbol Device:R_Small
- added R? (x4): 470, Resistor_SMD:R_0402_1005Metric, symbol Device:R_Small
- added R? (x2): 0R/1206, Resistor_SMD:R_1206_3216Metric_Pad1.30x1.75mm_HandSolder, symbol Device:R
- R?: value 100mR/1206 -> 50mR/1206
- R?: value 3k -> 5k
Connections:
- net OUT3_GND is gone; now on net GND: J?.2 (Pin_2)
- net +3.3V: now also J?.3 (Pin_3), JP?.2 (B), R?.1, R?.2, R?.2; no longer C?.1, C?.1, L?.2, R?.2, U?.6 (VDD)
- net +VDC: now also R?.1, R?.2, R?.2; no longer J?.1 (Pin_1), J?.1 (Pin_1)
- net ADC2: now also U?.1
- net GND: now also R?.1, C?.1, C?.2, J?.4 (Pin_4), R?.1, R?.1, R?.1, R?.1, R?.1, R?.1, R?.1, R?.1, R?.1, R?.1, R?.2; no longer C?.1, Q?.2 (S), Q?.2 (S), Q?.2 (S), Q?.2 (S), R?.1
- net I2C_SCL: now also J?.2 (Pin_2), R?.1
- net I2C_SDA: now also J?.1 (Pin_1), R?.1
- net IO8: no longer U?.14 (GPIO8)
- net IO9: no longer U?.15 (GPIO9/BOOT)
- net OUT1_CTRL: now also R?.2
- net OUT2_CTRL: now also R?.2
- net OUT2_GND: now also R?.1
- net OUT3_CTRL: now also R?.2
- net OUT3_PWR: now also J?.1 (Pin_1)
- net PWRIN_LED: now also Q?.3 (D), R?.2
- net SPK_PWM: now also C?.1, R?.1, U?.14 (GPIO8); no longer R?.2, U?.9 (MTMS/GPIO4/ADC1_CH4)
- net at Q?.1 (G), Q?.3 (D): now also R?.1 (x2)
- net at J?.2 (Pin_2), R?.2: now also R?.2, R?.2, R?.2
- net at Q?.1 (G), Q?.3 (D): now also Q?.1 (G), R?.1
- net at Q?.2 (S), R?.1: now also Q?.2 (S)
- net I2C_RST renamed SYS_RST
- new net: Q?.2 (S), R?.2 (x4)
- new net: C?.1, C?.2, JP?.1 (A), R?.2, U?.6 (VDD)
- new net: C?.1, C?.1, L?.2, R?.2, R?.2
- new net: J?.1 (Pin_1), R?.2
- new net BOOT_BUT1: U?.15 (GPIO9/BOOT)
- new net BUT2: U?.9 (MTMS/GPIO4/ADC1_CH4)
Other:
- note added: "A1 - 20V/V Imax=3A dVmax - 3.0/20 = 0.15V@3A R=U/I = 0.15/3 = 50mR P=I^2*R = 450mW"
- note added: "A3- 100V/V Imax=8A dVmax = 3.0/100 = 0.03V R=U/I = 0.03/8 = 3.75mR A1 - 20V/V dVmax - 3.0/20 = 0.15V@8A R = 3.75*5 = 18,75 -> 16.66mR P = I^2*R / 3 = 8*8*16.66m = 350mW"
- note added: "C127691 - I prefer this part everywhere to minimize bom"
- note added: "I know this looks spooky as hell but it's just a basic voltage divider, as PWM from ESP has way too large amplitude for this IC."
- note added: "So IO8 must be pulled-up on boot - this is done by voltage div near speaker amp."
- note added: "System has 3 points of current measurement: * Main Curr * OUT1 Curr * OUT2 Curr * OUT3 is NOT measured independently - therfore has lower power path impedance than the others OUT3, WS2812 and RGB currents must be calculated by substraction If OUT3&RGB are used, current measurements become ambigous with WS2812, we can either estimate current measurement, or calibrate system, by disabling everythin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"
- note added: "User interface"
- note added: "https://www.falstad.com/circuit/circuitjs.html?ctz=CQAgjCAMB0l3BWKsAsBOATCgbCjAOAdm0IRUjXxGwxCRQGY6BTAWjDACgxDbWtI4bIP7kQKKoMLjBYpIJhIAagHsANgBcAhgHNmnHSFb5BCMHxN0CUKJwBORy2GGPBDSChsJ4nAO6uhER5sQNt-dmIQd09jNw9bAAcjYKj4iJDnQQgFPwDyEUto2wAlEAxeGUECKgYMBRsxBmgmesVOADNkyKLROM8GJjBoJCbSAyMBcVwJuWsc8MnqmayXSFz00N7QtYBjLpCelMZaWjA2NCimjGwEBjBIG7QSW+zYSC5DDeP9q0lbBy2tREkxwniya06rFq4mceVh0IwzWQkAw9jy0NidH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"
- note removed: "https://www.falstad.com/circuit/circuitjs.html?ctz=CQAgjCAMB0l3BWKsAsBOATCgbCjAOAdm0IRUjXxGwxCRQGY6BTAWjDACgxDbWtI4bIP7kQKKoMJ1xgpIJhIAagHsANgBcAhgHNmnHSFb45YPiboEoUTgCcjFsMIeCGkFNbdxOAdxdCRHmwAmz92YhA3D2NXdxsAByMgyLjw4KdBCAVff3IRCyibACUQDF5ZQQIqBgwFazEGaCY6xU4AMySIwtFYjwYmMGgkRtIDIwFxXHGxBCtssImq6cznSBy0kJ6QtYBjTuDu5MZaWjA2NHAmyAQEBnJ0BGwwSCxkOC5DDeP9y0kbey2NREExwHkyaw6rBq4icuVh0MGtBgLzsuWhMToZm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"
- moved on the sheet: BZ?, C?, D?, J?, LS?, Q?, R?, SW?, U?

Commit message: pivoting to protoboard-matrix
Parts:
- removed BZ?: Buzzer_DNP, symbol Device:Buzzer
- removed C? (x5): 100n, Capacitor_SMD:C_0603_1608Metric, symbol Device:C_Small
- removed C? (x4): 10u, Capacitor_SMD:C_0603_1608Metric, symbol Device:C_Small
- removed C?: 330uF/6.3V, symbol Device:C_Polarized_Small_US
- removed C? (x2): TBD, Capacitor_SMD:C_0402_1005Metric, symbol Device:C_Small
- removed C?: 10n, Capacitor_SMD:C_0603_1608Metric, symbol Device:C_Small
- removed C? (x4): 100n, Capacitor_SMD:C_0402_1005Metric, symbol Device:C_Small
- removed C? (x2): 15p, Capacitor_SMD:C_0402_1005Metric, symbol Device:C_Small
- removed D?: SS54, symbol Device:D_Schottky
- removed J?: WS2812_OUT, symbol Connector_Generic:Conn_01x03
- removed J?: RGB_OUT, symbol Connector_Generic:Conn_01x04
- removed L?: TBD, symbol Device:L_Small
- removed L?: 2nH, symbol Device:L_Small
- removed LS?: Speaker, symbol Device:Speaker
- removed Q801: L8050QLT1G, symbol Device:Q_NPN_BEC
- removed Q? (x2): AO3400A, Package_TO_SOT_SMD:SOT-23, symbol Transistor_FET:AO3400A
- removed Q? (x5): 2N7002, Package_TO_SOT_SMD:SOT-23, symbol Transistor_FET:2N7002
- removed Q?: L8050QLT1G, Package_TO_SOT_SMD:SOT-23, symbol Device:Q_NPN_BEC
- removed R? (x9): 10k, Resistor_SMD:R_0402_1005Metric, symbol Device:R_Small
- removed R? (x4): 5k, Resistor_SMD:R_0603_1608Metric_Pad0.98x0.95mm_HandSolder, symbol Device:R_Small
- removed R? (x5): 470, Resistor_SMD:R_0402_1005Metric, symbol Device:R_Small
- removed R? (x3): 0R/1206, Resistor_SMD:R_1206_3216Metric_Pad1.30x1.75mm_HandSolder, symbol Device:R
- removed R? (x4): 2R/1206, Resistor_SMD:R_1206_3216Metric_Pad1.30x1.75mm_HandSolder, symbol Device:R
- removed R?: 0R/1206, Resistor_SMD:R_0402_1005Metric, symbol Device:R_Small
- removed SW?: B2, Byotta:SW_ALPS_SKRKAEE020, symbol Switch:SW_Push
- removed SW?: RST, Byotta:SW_ALPS_SKRKAEE020, symbol Switch:SW_Push
- removed SW?: BOOT/B1, Byotta:SW_ALPS_SKRKAEE020, symbol Switch:SW_Push
- removed U?: PCA9557PW, Package_SO:TSSOP-16_4.4x5mm_P0.65mm, symbol Interface_Expansion:PCA9557PW
- removed U?: ESP32-C3, Package_DFN_QFN:QFN-32-1EP_5x5mm_P0.5mm_EP3.45x3.45mm, symbol Espressif:ESP32-C3
- removed U? (x3): INA181, Package_TO_SOT_SMD:SOT-23-6, symbol Amplifier_Current:INA181
- removed Y?: 40MHz_3225, symbol Device:Crystal_GND24_Small
- added C1, C11, C6, C7: DNP, Capacitor_SMD:C_0402_1005Metric, symbol Device:C_Small
- added C19, C20, C21, C22, C3: 47uF/6.3V, Capacitor_SMD:C_1206_3216Metric, symbol Device:C_Small
- added C8: 100n, Capacitor_SMD:C_0402_1005Metric, symbol Device:C_Small
- added C9: 10u, Capacitor_SMD:C_0603_1608Metric, symbol Device:C_Small
- added D3: 1N5819WS, Diode_SMD:D_SOD-323, symbol Device:D_Schottky
- added H1, H2, H3, H4: SCR, MountingHole:MountingHole_3.2mm_M3_Pad_TopOnly, symbol Mechanical:MountingHole_Pad
- added J1: INA_STATE, Connector_PinHeader_2.54mm:PinHeader_1x04_P2.54mm_Vertical, symbol Connector_Generic:Conn_01x04
- added J4, J5, J6, J7: PROTO, Connector_PinSocket_2.54mm:PinSocket_2x10_P2.54mm_Vertical, symbol Connector_Generic:Conn_02x10_Top_Bottom
- added Q1: MMBT2222A, Buzzer_Beeper:Buzzer_TDK_PS1240P02BT_D12.2mm_H6.5mm, symbol Device:Q_NPN_BEC
- added Q10, Q13, Q14, Q15, Q16, Q19, Q5, Q6, Q9: MMBT2222A, Package_TO_SOT_SMD:SOT-23, symbol Device:Q_NPN_BEC
- added Q12, Q18, Q22, Q4, Q8: S9015, Package_TO_SOT_SMD:SOT-23, symbol Device:Q_PNP_BEC
- added Q21, Q23: AO3400A, Package_TO_SOT_SMD:SOT-23, symbol Transistor_FET:AO3400A
- added R1, R30, R42, R8: 15k, Resistor_SMD:R_0402_1005Metric, symbol Device:R_Small
- added R11, R12, R16, R2, R24, R3, R31, R33, R4, R43, R45, R49, R5, R59, R60, R7: 10k, Resistor_SMD:R_0402_1005Metric, symbol Device:R_Small
- added R13, R17, R29, R34, R50: 470, Resistor_SMD:R_0402_1005Metric, symbol Device:R_Small
- added R21, R22, R35, R39: 0R/1206, Resistor_SMD:R_1206_3216Metric_Pad1.30x1.75mm_HandSolder, symbol Device:R
- added RV1: 10k, Potentiometer_SMD:Potentiometer_Bourns_TC33X_Vertical, symbol Device:R_Potentiometer_Small
- added SW1: RST, Button_Switch_THT:SW_PUSH_6mm_H4.3mm, symbol Switch:SW_Push
- added SW2: BOOT/B1, Button_Switch_THT:SW_PUSH_6mm_H4.3mm, symbol Switch:SW_Push
- added SW3: B2, Button_Switch_THT:SW_PUSH_6mm_H4.3mm, symbol Switch:SW_Push
- added TP1, TP2, TP3, TP4, TP5, TP6: TestPoint, Connector_PinSocket_2.54mm:PinSocket_1x01_P2.54mm_Vertical, symbol Connector:TestPoint
- added U2: INA3221, Package_DFN_QFN:Texas_RGV_S-PVQFN-N16_EP2.1x2.1mm, symbol Power_Management:INA3221
- added U3: ESP32-C3-WROOM-02, Espressif:ESP32-C3-WROOM-02, symbol Espressif:ESP32-C3-WROOM-02
- C4: renamed from C?; footprint Capacitor_SMD:C_0603_1608Metric -> Capacitor_SMD:C_1206_3216Metric
- D1, D2: renamed from D?; value SS54 -> 1N5819WS; footprint (none) -> Diode_SMD:D_SOD-323
- D4, D5, D6, D7: renamed from D?; footprint LED_SMD:LED_0603_1608Metric -> LED_THT:LED_D3.0mm_IRBlack
- J11, J2, J3, J9: renamed from J?; footprint (none) -> TerminalBlock_WAGO:TerminalBlock_WAGO_236-402_1x02_P5.00mm_45Degree
- J13: renamed from J?; footprint (none) -> Connector_PinSocket_2.54mm:PinSocket_1x04_P2.54mm_Vertical
- JP1, JP2, JP3, JP4: renamed from JP?; footprint (none) -> Jumper:SolderJumper-2_P1.3mm_Open_TrianglePad1.0x1.5mm
- L1: renamed from L?; footprint (none) -> Inductor_SMD:L_2512_6332Metric
- R23, R26: renamed from R?; value 2R/1206 -> 0R/1206
- U5: renamed from U?; footprint (none) -> Package_SO:MSOP-8_3x3mm_P0.65mm
- gave numbers to parts that had none: 43
Connections:
- net +3.3V: now also C8.1, C9.1, J4.1 (Pin_1), J4.11 (Pin_11), J5.1 (Pin_1), J5.11 (Pin_11), Q22.2 (E), R2.2, R24.2, R3.2, R4.2, R5.2, U2.16 (VPU), U2.4 (VS), U3.1 (3V3); no longer D4.2 (A)
- net +VDC: now also J7.1 (Pin_1), J7.11 (Pin_11), Q10.3 (C), Q16.3 (C), Q5.3 (C), R30.2, R42.2, R8.2
- net BOOT_BUT1: now also C13.1, SW2.2, U3.8 (GPIO9)
- net BUT2: now also C18.1, SW3.2, U3.7 (GPIO8)
- net DTR: now also Q15.2 (E)
- net ESP_EN: now also Q14.3 (C), R24.1, SW1.2, U3.2 (EN/CHIP_PU)
- net GND: now also R51.1, C19.2, C20.2, C21.2, C22.2, C3.2, C8.2, C9.2, D3.2 (A), H1.1, H2.1, H3.1, H4.1, J4.10 (Pin_10), J4.20 (Pin_20), J5.10 (Pin_10), J5.20 (Pin_20), J6.10 (Pin_10), J6.20 (Pin_20), J7.10 (Pin_10), J7.20 (Pin_20), Q12.3 (C), Q18.3 (C), Q21.2 (S), Q23.2 (S), Q4.3 (C), Q8.3 (C), R11.1, R13.1, R16.1, R17.1, R21.2, R33.1, R34.1, R39.2, R45.1, R49.1, R59.1, SW1.1, SW2.1, SW3.1, U2.17 (EP), U2.3 (GND), U2.5 (A0), U3.19 (GND), U3.9 (GND); no longer J11.2 (Pin_2)
- net I2C_SCL: now also J4.6 (Pin_6), U2.6 (SCL), U3.4 (GPIO5/ADC2_CH0)
- net I2C_SDA: now also J4.7 (Pin_7), U2.7 (SDA), U3.5 (GPIO6)
- net IO8: now also J4.9 (Pin_9); no longer C18.1
- net IO9: now also Q15.3 (C); no longer C13.1
- net OUT1_GND: no longer J3.2 (Pin_2)
- net OUT1_PWR: no longer J3.1 (Pin_1)
- net OUT2_GND: now also R35.2; no longer J9.2 (Pin_2)
- net OUT2_PWR: no longer J9.1 (Pin_1)
- net OUT3_CTRL: now also C1.1, R7.2
- net OUT3_PWR: now also J7.12 (Pin_12); no longer J11.1 (Pin_1)
- net PWRIN_LED: now also Q1.3 (C), R1.2
- net RTS: now also Q14.2 (E)
- net SPK_PWM: now also U3.10 (GPIO10)
- net SYS_RST: now also J4.8 (Pin_8)
- net TARG_RX: now also U3.11 (GPIO20/U0RXD)
- net TARG_TX: now also R29.1, R60.1
- net VBUS: now also J6.1 (Pin_1), J6.11 (Pin_11)
- net at J8.A7 (D-), J8.B7 (D-): now also U3.13 (GPIO18/USB_D-)
- net at J8.A6 (D+), J8.B6 (D+): now also U3.14 (GPIO19/USB_D+)
- net at R46.2: now also Q19.2 (E)
- net at Q17.1 (G): now also Q16.2 (E), Q18.2 (E)
- net OUT1_SHUNTP: now reaches R23.1
- net OUT1_SHUNTP: now also U2.15 (IN+2)
- net OUT1_SNUNTN: now reaches R26.1
- net OUT1_SNUNTN: now also U2.14 (IN-2)
- net at J2.2 (Pin_2), R18.2, R19.2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: now also R22.2
- net at C14.1, C15.2, JP4.1 (A)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: now also RV1.1, RV1.2
- net at C2.1, L1.2, R10.2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: now also C19.1, C20.1, C21.1, C22.1, C3.1
- net at Q11.1 (G): now also Q10.2 (E), Q12.2 (E)
- net at R40.2: now also Q14.1 (B)
- net at Q7.1 (G): now also Q5.2 (E), Q8.2 (E)
- net at C16.1, R52.2: now also R50.1
- net SPK_OUTP: now reaches U5.5 (OUT+)
- net at Q2.1 (G), Q3.1 (G): now also Q1.2 (E), Q4.2 (E)
- net at L1.1, U1.2 (OUT): now also D3.1 (K)
- net SPK_OUTN: now reaches U5.8 (OUT-)
- net at R41.2: now also Q15.1 (B)
- net OUTR: now reaches Q20.3 (D)
- net OUTR_CTRL renamed GATE_R
- new net: J3.1 (Pin_1), TP1.1
- new net: J3.2 (Pin_2), TP2.1
- new net: Q6.2 (E), R13.2
- new net: C1.2, Q6.1 (B), R11.2, R7.1
- new net: C7.2, Q13.1 (B), R31.1, R33.2
- new net: J9.2 (Pin_2), TP4.1
- new net: Q5.1 (B), Q8.1 (B), Q9.3 (C), R8.1
- new net: Q1.1 (B), Q4.1 (B), Q6.3 (C), R1.1
- new net: R50.2, RV1.3
- new net: J9.1 (Pin_1), TP3.1
- new net: J1.1 (Pin_1), R5.1, U2.10 (PV)
- new net: J1.2 (Pin_2), R4.1, U2.9 (CRITICAL)
- new net: J1.3 (Pin_3), R3.1, U2.8 (WARNING)
- new net: J1.4 (Pin_4), R2.1, U2.13 (TC)
- new net: Q13.2 (E), R34.2
- new net: J11.1 (Pin_1), TP5.1
- new net: Q16.1 (B), Q18.1 (B), Q19.3 (C), R42.1
- new net: J11.2 (Pin_2), TP6.1
- new net: C11.2, Q19.1 (B), R43.1, R45.2
- new net: D4.2 (A), Q22.3 (C)
- new net: C6.2, Q9.1 (B), R12.1, R16.2
- new net: Q10.1 (B), Q12.1 (B), Q13.3 (C), R30.1
- new net: Q9.2 (E), R17.2
- new net: R29.2, U3.12 (GPIO21/U0TXD)
- new net: Q22.1 (B), R60.2
- new net GATE_B: Q23.1 (G), R59.2
- new net GATE_G: Q21.1 (G), R49.2
- new net GATE_O1: C6.1, R12.2
- new net GATE_O2: C7.1, R31.2
- new net GATE_O3: C11.1, R43.2
- new net IO0: J4.2 (Pin_2), U3.18 (GPIO0/ADC1_CH0/XTAL_32K_P)
- new net IO1: J4.3 (Pin_3), U3.17 (GPIO1/ADC1_CH1/XTAL_32K_N)
- new net IO2: J4.5 (Pin_5), U3.16 (GPIO2/ADC1_CH2)
- new net IO3: J4.4 (Pin_4), U3.15 (GPIO3/ADC1_CH3)
- new net IO4: U3.3 (GPIO4/ADC1_CH4)
- new net IO7: U3.6 (GPIO7)
- new net OUT2_SHUNTP: R35.1, U2.2 (IN+3)
- new net OUT2_SNUNTN: R39.1, U2.1 (IN-3)
- new net OUTB: J7.19 (Pin_19), Q23.3 (D)
- new net OUTG: Q21.3 (D)
- new net VIN_SHUNTN: R22.1, U2.11 (IN-1)
- new net VIN_SHUNTP: R21.1, U2.12 (IN+1)
- no-connect marks 10 -> 48
Other:
- note added: "Protoboard area"
- note added: "https://www.falstad.com/circuit/circuitjs.html?ctz=CQAgjCAMB0l3BWKsAsBOATCgbCjAOAdm0IRUjXxGwxCRQGY6BTAWjDACgxDbWHsVMNkgh+gkCiqjCk0eTpRkSAGoB7ADYAXAIYBzZpwBOY-KOGjWZkA0golYBPE4B3MRkhCRY2-YtROAAcfOxtQ-lD-CFFITgAlECxRX0SEbESsJXlk6CYY5U4AMxD7FPEqFIYmMGgkBmhSTj0fCRx7croCLNcWqgIqDv9Ytwi-b0HvWIBjErD2lMZaWjA2CrQGsDNHQkI0MBw05DguZtHJBj4UhC6Y416bD3u2h1iAZXAUUsekh-yIQp0GgAzswlBgmokFFV0hhDuR8rEtGIwF0MLx3J5Eu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"
- note removed: "$0.20"
- note removed: "1.8V@40Vin"
- note removed: "A1 - 20V/V Imax=3A dVmax - 3.0/20 = 0.15V@3A R=U/I = 0.15/3 = 50mR P=I^2*R = 450mW"
- note removed: "A3- 100V/V Imax=8A dVmax = 3.0/100 = 0.03V R=U/I = 0.03/8 = 3.75mR A1 - 20V/V dVmax - 3.0/20 = 0.15V@8A R = 3.75*5 = 18,75 -> 16.66mR P = I^2*R / 3 = 8*8*16.66m = 350mW"
- note removed: "For Hfe in range 150-300: Ibe = (3.3V - 0.7V)/R? Assume Ibe=10uA R? = 2.7/10uA = 2.7*100k = 270k for Ibe=10uA Ice range is [1.5-3]mA Assume VDC=5V, Rgs=10k Ugs = 10k*1mA = 10V"
- note removed: "https://www.falstad.com/circuit/circuitjs.html?ctz=CQAgjCAMB0l3BWKsAsBOATCgbCjAOAdm0IRUjXxGwxCRQGY6BTAWjDACgxDbWtI4bIP7kQKKoMLjBYpIJhIAagHsANgBcAhgHNmnHSFb5BCMHxN0CUKJwBORy2GGPBDSChsJ4nAO6uhER5sQNt-dmIQd09jNw9bAAcjYKj4iJDnQQgFPwDyEUto2wAlEAxeGUECKgYMBRsxBmgmesVOADNkyKLROM8GJjBoJCbSAyMBcVwJuWsc8MnqmayXSFz00N7QtYBjLpCelMZaWjA2NCimjGwEBjBIG7QSW+zYSC5DDeP9q0lbBy2tREkxwniya06rFq4mceVh0IwzWQkAw9jy0NidH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"
- note removed: "https://www.falstad.com/circuit/circuitjs.html?ctz=CQAgjCAMB0l3BWKsDMCBMAOAbNymwAWBTTQzAThG3RCUJToFMBaMMAKDAHZaX1CkcHhD9BIclBDcQWWZilCYSAGoB7ADYAXAIYBzJhz2jMQhn1N05SjgCcTQsCJaWUkQlLDxIHAF5S3D0cRWgATJgAzHQBXbRZfJgA7JlsOAHcHYSE2bmwsqHTRHjzAzNKfAAci3JBSnLynR0UOLVEUWkInTM68pv5uaGxSTBQUbkx0SBJ0WhgUdjhCLF5JhEh0GTwhcKjYrUKXMzgy9wL7FnaJLskeqQ3vQpuu4qvewuDsy0aCjKE611OPgASuAaqUwBRaDMglJxChoIwlMgEBwItUSqcxH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"
- moved on the sheet: D4, D6, D7, J10, J11, J3, J9, JP2, JP3, Q11, Q17, Q20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
