File: cringenode.kicad_sch (KiCad schematic)
At the start: 142 parts, among them J1 INA_STATE, J10 PROG_HEADER, J11 PWR_OUT_3, J13 OLED, J2 PWR_IN, J3 PWR_OUT_1, J4 PROTO, J5 PROTO, J6 PROTO, J7 PROTO, J8 USB_C_Receptacle_USB2.0, J9 PWR_OUT_2, Q1 MMBT2222A, Q10 MMBT2222A, Q11 WST03P06, Q12 S9015, Q13 MMBT2222A, Q14 MMBT2222A, Q15 MMBT2222A, Q16 MMBT2222A, Q17 WST03P06, Q18 S9015, Q19 MMBT2222A, Q2 WST03P06, Q20 AO3400A, Q21 AO3400A, Q22 S9015, Q23 AO3400A, Q3 WST03P06, Q4 S9015, Q5 MMBT2222A, Q6 MMBT2222A, Q7 WST03P06, Q8 S9015, Q9 MMBT2222A, SW1 RST, SW2 BOOT/B1, SW3 B2, U1 XL1509, U2 INA3221, U3 ESP32-C3-WROOM-02, U5 PAM8302AAD

Commit message: finish this unholy abomination
Parts:
- removed C11, C6, C7: DNP, Capacitor_SMD:C_0402_1005Metric, symbol Device:C_Small
- removed D4: LED_0603, LED_THT:LED_D3.0mm_IRBlack, symbol Device:LED
- removed J1: INA_STATE, Connector_PinHeader_2.54mm:PinHeader_1x04_P2.54mm_Vertical, symbol Connector_Generic:Conn_01x04
- removed J10: PROG_HEADER, Connector_PinHeader_2.54mm:PinHeader_1x08_P2.54mm_Vertical, symbol Connector_Generic:Conn_01x08
- removed J11: PWR_OUT_3, TerminalBlock_WAGO:TerminalBlock_WAGO_236-402_1x02_P5.00mm_45Degree, symbol Connector:Screw_Terminal_01x02
- removed J13: OLED, Connector_PinSocket_2.54mm:PinSocket_1x04_P2.54mm_Vertical, symbol Connector_Generic:Conn_01x04
- removed J2: PWR_IN, TerminalBlock_WAGO:TerminalBlock_WAGO_236-402_1x02_P5.00mm_45Degree, symbol Connector:Screw_Terminal_01x02
- removed J3: PWR_OUT_1, TerminalBlock_WAGO:TerminalBlock_WAGO_236-402_1x02_P5.00mm_45Degree, symbol Connector:Screw_Terminal_01x02
- removed J4, J5, J6, J7: PROTO, Connector_PinSocket_2.54mm:PinSocket_2x10_P2.54mm_Vertical, symbol Connector_Generic:Conn_02x10_Top_Bottom
- removed J9: PWR_OUT_2, TerminalBlock_WAGO:TerminalBlock_WAGO_236-402_1x02_P5.00mm_45Degree, symbol Connector:Screw_Terminal_01x02
- removed Q10, Q13, Q16, Q19, Q5, Q9: MMBT2222A, Package_TO_SOT_SMD:SOT-23, symbol Device:Q_NPN_BEC
- removed Q11, Q17, Q7: WST03P06, Package_TO_SOT_SMD:SOT-23, symbol Critbit_lib:WST03P06
- removed Q12, Q18, Q22, Q8: S9015, Package_TO_SOT_SMD:SOT-23, symbol Device:Q_PNP_BEC
- removed R12, R16, R31, R33, R43, R45, R60: 10k, Resistor_SMD:R_0402_1005Metric, symbol Device:R_Small
- removed R15, R21, R22, R23, R26, R32, R35, R39, R44: 0R/1206, Resistor_SMD:R_1206_3216Metric_Pad1.30x1.75mm_HandSolder, symbol Device:R
- removed R17, R46, R51: 470, Resistor_SMD:R_0402_1005Metric, symbol Device:R_Small
- removed R30, R42, R8: 15k, Resistor_SMD:R_0402_1005Metric, symbol Device:R_Small
- added C12: 10u, Capacitor_SMD:C_0603_1608Metric, symbol Device:C_Small
- added C13, C21: 100n, Capacitor_SMD:C_0402_1005Metric, symbol Device:C_Small
- added D5, D8: LED_0603, LED_SMD:LED_0603_1608Metric_Pad1.05x0.95mm_HandSolder, symbol Device:LED
- added J1: IN+, Critbit_lib:DG235-5.0, symbol Connector:Screw_Terminal_01x01
- added J10, J11, J12, J6, J7, J9: TERM_BLOCK, Critbit_lib:DG235-5.0, symbol Connector:Screw_Terminal_01x01
- added J2: IN-, Critbit_lib:DG235-5.0, symbol Connector:Screw_Terminal_01x01
- added J3: Proto_matrix_14x9+7, Critbit_lib:Proto_matrix_14x9+7, symbol Critbit_lib:Proto_matrix_14x9+7
- added J5: Lichtenprog_conn, Critbit_lib:Lichtenprog, symbol Critbit_lib:Lichtenprog_conn
- added J8: INA_STA, Connector_PinHeader_2.54mm:PinHeader_2x02_P2.54mm_Vertical, symbol Connector_Generic:Conn_02x02_Odd_Even
- added JP2, JP3: SolderJumper_3_Open, Jumper:SolderJumper-3_P2.0mm_Open_TrianglePad1.0x1.5mm_NumberLabels, symbol Jumper:SolderJumper_3_Open
- added R20, R37: 10k, Resistor_SMD:R_0402_1005Metric, symbol Device:R_Small
- added SW4: B3, Button_Switch_SMD:SW_SPST_FSMSM, symbol Switch:SW_Push
- added TP1, TP5, TP6, TP9: INA_PAD, TestPoint:TestPoint_Pad_D2.5mm, symbol Connector:TestPoint
- added TP2: GND_PAD, TestPoint:TestPoint_Pad_D2.5mm, symbol Connector:TestPoint
- C1: renamed from C2; footprint Capacitor_SMD:C_0603_1608Metric -> Capacitor_SMD:C_0402_1005Metric
- C8: renamed from C5; footprint Capacitor_SMD:C_0603_1608Metric -> Capacitor_SMD:C_0402_1005Metric
- D4: renamed from D5; footprint LED_THT:LED_D3.0mm_IRBlack -> LED_SMD:LED_0603_1608Metric_Pad1.05x0.95mm_HandSolder
- D6, D7: footprint LED_THT:LED_D3.0mm_IRBlack -> LED_SMD:LED_0603_1608Metric_Pad1.05x0.95mm_HandSolder
- L1: value L -> 47uH/2A; footprint Inductor_SMD:L_2512_6332Metric -> Inductor_SMD:L_Abracon_ASPI-0630LR; JLC (none) -> C149588
- Q1: footprint Buzzer_Beeper:Buzzer_TDK_PS1240P02BT_D12.2mm_H6.5mm -> Package_TO_SOT_SMD:SOT-23
- R12: renamed from R19; value 50mR/1206 -> 0R/1206
- R18: renamed from R36; footprint Resistor_SMD:R_0603_1608Metric_Pad0.98x0.95mm_HandSolder -> Resistor_SMD:R_0402_1005Metric
- R19: renamed from R37; footprint Resistor_SMD:R_0603_1608Metric_Pad0.98x0.95mm_HandSolder -> Resistor_SMD:R_0402_1005Metric
- R29: value 470 -> DNP
- R32: renamed from R52; value 470 -> DNP
- R34: value 470 -> 10k
- SW1, SW2, SW3: footprint Button_Switch_THT:SW_PUSH_6mm_H4.3mm -> Button_Switch_SMD:SW_SPST_FSMSM
- TP10: renamed from TP5; value TestPoint -> CON_PAD; footprint Connector_PinSocket_2.54mm:PinSocket_1x01_P2.54mm_Vertical -> MountingHole:MountingHole_2.7mm_M2.5_DIN965_Pad
- TP11: renamed from TP6; value TestPoint -> CON_PAD; footprint Connector_PinSocket_2.54mm:PinSocket_1x01_P2.54mm_Vertical -> MountingHole:MountingHole_2.7mm_M2.5_DIN965_Pad
- TP3: renamed from TP1; value TestPoint -> CON_PAD; footprint Connector_PinSocket_2.54mm:PinSocket_1x01_P2.54mm_Vertical -> MountingHole:MountingHole_2.7mm_M2.5_DIN965_Pad
- TP4: renamed from TP2; value TestPoint -> CON_PAD; footprint Connector_PinSocket_2.54mm:PinSocket_1x01_P2.54mm_Vertical -> MountingHole:MountingHole_2.7mm_M2.5_DIN965_Pad
- TP7: renamed from TP3; value TestPoint -> CON_PAD; footprint Connector_PinSocket_2.54mm:PinSocket_1x01_P2.54mm_Vertical -> MountingHole:MountingHole_2.7mm_M2.5_DIN965_Pad
- TP8: renamed from TP4; value TestPoint -> CON_PAD; footprint Connector_PinSocket_2.54mm:PinSocket_1x01_P2.54mm_Vertical -> MountingHole:MountingHole_2.7mm_M2.5_DIN965_Pad
- renumbered C8 to C10, C9 to C11, C12 to C14, C13 to C15, C18 to C16, C14 to C17, C15 to C18, C16 to C19, C3 to C2, C17 to C20, C19 to C3, C20 to C4, C21 to C5, C22 to C6, C4 to C7, C1 to C9, J8 to J4, JP2 to JP4, JP3 to JP5, JP4 to JP6, Q15 to Q10, Q20 to Q4, Q4 to Q5, Q21 to Q7, Q23 to Q8, Q14 to Q9, R18 to R1, R13 to R10, R49 to R11, R9 to R13, R59 to R14, R24 to R15, R27 to R16, R28 to R17, R20 to R2, R40 to R21, R41 to R22, R2 to R23, R3 to R24, R4 to R25, R5 to R26, R25 to R27, R38 to R28, R6 to R3, R50 to R31, R54 to R33, R56 to R35, R57 to R36, R1 to R4, R10 to R5, R47 to R6, R14 to R8, R11 to R9, U3 to U2, U2 to U3, U5 to U4
Connections:
- net IO9 is gone; now on net IO9/BOOT_BUT1: Q10.3 (C)
- net OUT2_GND is gone; now on an unnamed net: R28.1
- net OUT2_SHUNTP is gone; now on net VIN_SHUNTP: U3.2 (IN+3)
- net OUT2_SNUNTN is gone; now on net VIN_SHUNTN: U3.1 (IN-3)
- net OUT3_CTRL is gone; now on net IO7/GATE_IN: C9.1, R7.2
- net STA_LED is gone; now on net IO7/GATE_IN: D7.2 (A)
- net +3.3V: now also C12.1, C13.2, J3.A3, J3.B1, R20.2; no longer U4.1 (~{SD})
- net +VDC: now also Q2.2 (S), Q3.2 (S), J3.J4; no longer R13.2
- net DTR: now also J5.3 (DTR)
- net GATE_B: now also J3.C1
- net GATE_G: now also J3.D1
- net GATE_O1: now also J3.H1
- net GATE_O2: now also J3.G1
- net GATE_O3: now also J3.F1
- net GATE_R: now also J3.E1
- net GND: now also C20.1, R13.1, R32.1, C12.2, C13.1, C21.2, J3.A1, J3.A2, J3.D14, J3.E14, J3.F14, J3.G14, J3.H14, J3.I14, J5.6 (GND), J5.7 (GND), JP2.1 (A), R37.1, SW4.1, TP2.1; no longer H3.1, H4.1, R1.1, R2.1, R27.2, R28.2
- net IO0: now also J3.A6
- net IO1: now also J3.A7
- net IO2: now also J3.A8
- net OUT1_PWR: now also J3.J1
- net OUT2_PWR: now also J3.J2
- net OUT3_PWR: now also J3.J3
- net OUTB: now also J3.J7
- net OUTG: now also J3.J6
- net OUTR: now also J3.J5
- net RTS: now also J5.2 (RTS)
- net SPK_OUTN: now also J3.C14
- net SPK_OUTP: now also J3.B14
- net TARG_RX: now also J5.5 (PROG_TX)
- net TARG_TX: now also U2.12 (GPIO21/U0TXD), J5.4 (PROG_RX); no longer R29.1
- net VBUS: now also D8.2 (A), J3.I1
- net VIN_SHUNTN: now also JP3.2 (C); no longer U3.11 (IN-1)
- net VIN_SHUNTP: now also JP2.2 (C); no longer U3.12 (IN+1)
- net DCDC_L: now reaches C1.1, C2.1, C3.1, C4.1, C5.1, C6.1, L1.2, R3.2, R5.2
- net TERM1: now reaches TP3.1
- net TERM1: now also J6.1 (Pin_1)
- net TERM2: now reaches TP4.1
- net TERM2: now also J7.1 (Pin_1)
- net at JP5.1 (A): now also J5.8 (5V)
- net at R1.2, R2.2: now also Q2.3 (D), Q3.3 (D), JP3.3 (B); no longer R12.2
- net 3V3_SPK: now reaches C17.1, C18.2, JP6.1 (A), U4.6 (VDD)
- net 3V3_SPK: now also U4.1 (~{SD}); no longer RV1.1, RV1.2
- net TERM4: now reaches TP8.1
- net TERM4: now also J10.1 (Pin_1)
- net at R31.2, RV1.3: now also R29.1
- net TERM3: now reaches TP7.1
- net TERM3: now also J9.1 (Pin_1)
- net at R26.1, U3.10 (PV): now also J8.1 (Pin_1)
- net at R25.1, U3.9 (CRITICAL): now also J8.2 (Pin_2)
- net at R24.1, U3.8 (WARNING): now also J8.4 (Pin_4)
- net at R23.1, U3.13 (TC): now also J8.3 (Pin_3)
- net at R34.2: now also D5.1 (K)
- net TERM5: now reaches TP10.1
- net TERM5: now also J11.1 (Pin_1)
- net TERM6: now reaches TP11.1
- net TERM6: now also J12.1 (Pin_1)
- net DCDC_OUT: now reaches D3.1 (K), L1.1, U1.2 (OUT)
- net at JP4.1 (A): now also J5.1 (VDD)
- net IO10/SPK_PWM: now reaches R29.2
- net IO10/SPK_PWM: now also RV1.1, RV1.2, U2.10 (GPIO10), J3.A14; no longer U2.12 (GPIO21/U0TXD)
- net USBDM: now reaches J4.A7 (D-), J4.B7 (D-), U2.13 (GPIO18/USB_D-)
- net USBDP: now reaches J4.A6 (D+), J4.B6 (D+), U2.14 (GPIO19/USB_D+)
- net BOOT_BUT1 renamed IO9/BOOT_BUT1
- net IO9/BOOT_BUT1: now also J3.A13
- net BUT2 renamed IO8/BUT2
- net IO8/BUT2: now also J3.A12, R20.1
- net I2C_SCL renamed IO5/SCL
- net IO5/SCL: now also J3.A4
- net I2C_SDA renamed IO6/SDA
- net IO6/SDA: now also J3.A5
- net IO3 renamed IO3/BUT3
- net IO3/BUT3: now also C21.1, J3.A9, SW4.2
- net IO4 renamed IO4/LED
- net IO4/LED: now also D5.2 (A), J3.A10
- net IO7 renamed IO7/GATE_IN
- net IO7/GATE_IN: now also J3.A11
- net OUT1_GND: no longer names the net of R27.1
- net OUT1_GND: now also U3.12 (IN+1), TP1.1
- net OUT1_SHUNTP: no longer names the net of U3.15 (IN+2)
- net OUT1_SHUNTP: now also TP6.1
- net OUT1_SNUNTN: no longer names the net of U3.14 (IN-2)
- net OUT1_SNUNTN: now also R28.2, TP9.1
- net PWRIN_LED renamed V_IN
- net V_IN: now also R1.1, R2.1, J1.1 (Pin_1), JP2.3 (B); no longer Q2.3 (D), Q3.3 (D)
- removed net SPK_PWM: C20.1, R32.1, U2.10 (GPIO10)
- new net: R27.2, TP5.1, U3.11 (IN-1)
- new net: D8.1 (K), R37.2
- new net HACHET_FILL_NC: H3.1, H4.1
- new net V_IN_GND: J2.1 (Pin_1), JP3.1 (A), R12.2, R13.2
- no-connect marks 48 -> 2
Other:
- added sheet High side load switch (hi_side_sw.kicad_sch)
- added sheet High side load switch1 (hi_side_sw.kicad_sch)
- added sheet High side load switch2 (hi_side_sw.kicad_sch)
- note added: "OLED"
- note added: "Simulation of power switches: https://www.falstad.com/circuit/circuitjs.html?ctz=CQAgjCAMB0l3BWKsAsBOATCgbCjAOAdm0IRUjXxGwxCRQGY6BTAWjDACgxDbWHsVMNkgh+gkCiqjCk0eTpRkSAGoB7ADYAXAIYBzZpwBOY-KOGjWZkA0golYBPE4B3MRkhCRY2-YtROAAcfOxtQ-lD-CFFITgAlECxRX0SEbESsJXlk6CYY5U4AMxD7FPEqFIYmMGgkBmhSTj0fCRx7croCLNcWqgIqDv9Ytwi-b0HvWIBjErD2lMZaWjA2CrQGsDNHQkI0MBw05DguZtHJBj4UhC6Y416bD3u2h1iAZXAUUsekh-yIQp0GgAzswlB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"
- note added: "System has 3 points of current measurement - all are low side to ensure compatibility with 26V+ systems directly to INA3221: * VIN routed to proto matrix: * OUT1 * OUT2 Low side of outputs may be connected to OUT1/OUT2. Obvoiusly, it can't work with low side switches, in case of these, only cumulative output power may be measured. 7 load switches (MOSFET based) on the system High side (PMOSes): *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"
- note added: "This will be prolly a very noisy voltage rail due to shitty DC/DC. Oh well, let's see how it works."
- note added: "Transistors used in this project (all sot23) WST03P06 PMOS, 3.5A, 60VDS, 20VGS, 88Rds AO3400A NMOS, 5.7A, 30VDS, 12VGS, 48Rds MMBT2222A NPN, 0.6A, 40VCE, 75VCB S9015 PNP, 0.1A, 45VCE, 50VCB Diode: 1N5819WS 40V, 1A, SOD323"
- note added: "dUmax = 163.8mV Iin_max = 6A => Rin=25mR Iout_max = 3A => Rout=50mR"
- note removed: "CHECK PINOUT!!!!!!"
- note removed: "I know this looks spooky as hell but it's just a basic voltage divider, as PWM from ESP has way too large amplitude for this IC."
- note removed: "So IO8 must be pulled-up on boot - this is done by voltage div near speaker amp."
- note removed: "System has 3 points of current measurement: * Main Curr * OUT1 Curr * OUT2 Curr * OUT3 is NOT measured independently - therfore has lower power path impedance than the others OUT3, WS2812 and RGB currents must be calculated by substraction If OUT3&RGB are used, current measurements become ambigous with WS2812, we can either estimate current measurement, or calibrate system, by disabling everythin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"
- note removed: "https://www.falstad.com/circuit/circuitjs.html?ctz=CQAgjCAMB0l3BWKsAsBOATCgbCjAOAdm0IRUjXxGwxCRQGY6BTAWjDACgxDbWHsVMNkgh+gkCiqjCk0eTpRkSAGoB7ADYAXAIYBzZpwBOY-KOGjWZkA0golYBPE4B3MRkhCRY2-YtROAAcfOxtQ-lD-CFFITgAlECxRX0SEbESsJXlk6CYY5U4AMxD7FPEqFIYmMGgkBmhSTj0fCRx7croCLNcWqgIqDv9Ytwi-b0HvWIBjErD2lMZaWjA2CrQGsDNHQkI0MBw05DguZtHJBj4UhC6Y416bD3u2h1iAZXAUUsekh-yIQp0GgAzswlBgmokFFV0hhDuR8rEtGIwF0MLx3J5Eu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"
- moved on the sheet: C10, C11, C14, C15, C16, C9, D4, D6, D7, J4, JP4, JP5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
