File: MOSNode.kicad_sch (KiCad schematic)
At the start: 118 parts, among them J1 IN+, J10 TERM_BLOCK, J11 TERM_BLOCK, J12 TERM_BLOCK, J2 IN-, J3 Proto_matrix_14x9+7, J4 USB_C_Receptacle_USB2.0, J5 Lichtenprog_conn, J6 TERM_BLOCK, J7 TERM_BLOCK, J8 INA_STA, J9 TERM_BLOCK, Q1 MMBT2222A, Q10 MMBT2222A, Q2 WST03P06, Q3 WST03P06, Q4 AO3400A, Q5 S9015, Q6 MMBT2222A, Q7 AO3400A, Q8 AO3400A, Q9 MMBT2222A, SW1 RST, SW2 BOOT/B1, SW3 B2, SW4 B3, U1 XL1509, U2 ESP32-C3-WROOM-02, U3 INA3221, U4 PAM8302AAD

Commit message: replace audio with IOexp + PD controller, project rename
Parts:
- removed C3: 47uF/6.3V, Capacitor_SMD:C_1206_3216Metric, symbol Device:C_Small
- removed R16, R17: 470, Resistor_SMD:R_0402_1005Metric, symbol Device:R_Small
- removed RV1: 10k, Potentiometer_SMD:Potentiometer_Bourns_TC33X_Vertical, symbol Device:R_Potentiometer_Small
- removed U4: PAM8302AAD, Package_SO:MSOP-8_3x3mm_P0.65mm, symbol Amplifier_Audio:PAM8302AAD
- added C25: 200p, Capacitor_SMD:C_0402_1005Metric, symbol Device:C_Small
- added C3: C_THT, Capacitor_THT:CP_Radial_D10.0mm_P7.50mm, symbol Device:C_Polarized
- added R30, R38: 1k, Resistor_SMD:R_0402_1005Metric, symbol Device:R_Small
- added TP12, TP13, TP14, TP15, TP16, TP17, TP18, TP19, TP20: IOPAD, TestPoint:TestPoint_Pad_D1.0mm, symbol Connector:TestPoint
- added U4: PCA9557PW, Package_SO:TSSOP-16_4.4x5mm_P0.65mm, symbol Interface_Expansion:PCA9557PW
- added U5: FUSB302B01MPX, Package_DFN_QFN:WQFN-14-1EP_2.5x2.5mm_P0.5mm_EP1.45x1.45mm, symbol Interface_USB:FUSB302B01MPX
- C1: value 10n -> 200p; LCSC (none) -> C1530
- C10, C13, C14, C15, C16, C18, C21, C8: LCSC (none) -> C1525
- C11, C12: footprint Capacitor_SMD:C_0603_1608Metric -> Capacitor_SMD:C_0402_1005Metric; LCSC (none) -> C15525
- C17, C19: value 10u -> 100n; footprint Capacitor_SMD:C_0603_1608Metric -> Capacitor_SMD:C_0402_1005Metric; LCSC (none) -> C1525
- C2, C4, C5, C6, C7: LCSC C19702 -> C12891
- C20: value 10u -> 200p; footprint Capacitor_SMD:C_0603_1608Metric -> Capacitor_SMD:C_0402_1005Metric; LCSC (none) -> C1530
- C9: value DNP -> 200p; LCSC (none) -> C1530
- JP6: value SPK_ENA -> FUSB_INT_IO3
- Q1, Q10, Q6, Q9: LCSC (none) -> C8512
- R10: value 470 -> 1k; LCSC C25117 -> (none)
- R11, R14, R15, R20, R21, R22, R23, R24, R25, R26, R33, R34, R35, R36, R37, R4, R5, R6, R7, R8, R9: LCSC C25117 -> (none)
- R29, R32: value DNP -> 1k; LCSC C25117 -> (none)
- R31: value 470 -> 3k; LCSC C25117 -> (none)
Connections:
- net +3.3V: now also C17.2, C18.2, R29.2, R31.2, R32.2, R30.2, R38.2, U4.16 (VDD), U5.3 (VDD), U5.4 (VDD); no longer JP6.2 (B)
- net +VDC: now also Q2.3 (S), Q3.3 (S); no longer Q2.2 (S), Q3.2 (S)
- net DCDC_L: now also C3.1
- net GND: now also C17.1, C19.1, C20.2, C25.2, C3.2, U4.5 (A2), U4.8 (VSS), U5.15 (GND), U5.8 (GND), U5.9 (GND); no longer C17.2, C20.1, R32.1
- net IO3/BUT3: now also JP6.2 (B)
- net IO5/SCL: now also U4.1 (SCL), U5.6 (SCL)
- net IO6/SDA: now also U4.2 (SDA), U5.7 (SDA)
- net VBUS: now also C19.2, U5.12 (VCONN), U5.13 (VCONN), U5.2 (VBUS)
- net VIN_DC: now reaches C7.1, C8.1, D1.1 (K), D2.1 (K), U1.1 (VIN)
- net V_IN_MOSFETS: now reaches JP3.3 (B), R1.2, R2.2
- net V_IN_MOSFETS: now also Q2.2 (D), Q3.2 (D); no longer Q2.3 (D), Q3.3 (D)
- net at R29.1: now also TP18.1, U4.15 (~{RESET}); no longer R31.2
- net CC1: now reaches J4.A5 (CC1)
- net CC1: now also C20.1, TP19.1, U5.10 (CC1), U5.11 (CC1)
- net CC2: now reaches J4.B5 (CC2)
- net CC2: now also C25.1, TP20.1, U5.1 (CC2), U5.14 (CC2)
- removed net 3V3_SPK: C17.1, C18.2, JP6.1 (A)
- net IO10/SPK_PWM renamed IO10
- net IO10: no longer R29.2
- net OUTB renamed SINK_B
- net OUTG renamed SINK_G
- net OUTR renamed SINK_R
- net SPK_OUTN renamed EXT_IO2
- net EXT_IO2: now also U4.9 (IO2)
- net SPK_OUTP renamed EXT_IO1
- net EXT_IO1: now also U4.7 (IO1)
- new net: R32.1, U4.4 (A1)
- new net: R38.1, U4.3 (A0)
- new net: JP6.1 (A), R31.1, U5.5 (INT_N)
- new net EXT_IO0: R30.1, TP12.1, U4.6 (IO0)
- new net EXT_IO3: TP13.1, U4.10 (IO3)
- new net EXT_IO4: TP14.1, U4.11 (IO4)
- new net EXT_IO5: TP15.1, U4.12 (IO5)
- new net EXT_IO6: TP16.1, U4.13 (IO6)
- new net EXT_IO7: TP17.1, U4.14 (IO7)
Other:
- note added: "ADDR: 0011 A2 A1 A0 24-31 / 0x18-0x1F def. 27/0x1B"
- note added: "ADDR: 0x3C"
- note added: "ADDR: 10000XX (A0 grounded - XX=00) 64 / 0x40"
- note added: "Simulation of power switches (Link)"
- note removed: "Simulation of power switches: https://www.falstad.com/circuit/circuitjs.html?ctz=CQAgjCAMB0l3BWKsAsBOATCgbCjAOAdm0IRUjXxGwxCRQGY6BTAWjDACgxDbWHsVMNkgh+gkCiqjCk0eTpRkSAGoB7ADYAXAIYBzZpwBOY-KOGjWZkA0golYBPE4B3MRkhCRY2-YtROAAcfOxtQ-lD-CFFITgAlECxRX0SEbESsJXlk6CYY5U4AMxD7FPEqFIYmMGgkBmhSTj0fCRx7croCLNcWqgIqDv9Ytwi-b0HvWIBjErD2lMZaWjA2CrQGsDNHQkI0MBw05DguZtHJBj4UhC6Y416bD3u2h1iAZXAUUsekh-yIQp0GgAzswlB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"
- moved on the sheet: C2, H1, H2, H3, H4, J3

Commit message: production
Parts:
- C10, C13, C14, C15, C16, C17, C18, C19, C21, C8: LCSC C1525 -> C307331
- C2, C4, C5, C6, C7: LCSC C12891 -> C96123
- C3, H1, H2, H3, H4, J1, J10, J11, J12, J2, J3, J5, J6, J7, J8, J9, JP1, JP2, JP3, JP4, JP5, JP6, SW1, SW2, SW3, SW4, TP1, TP10, TP11, TP12, TP13, TP14, TP15, TP16, TP17, TP18, TP19, TP2, TP20, TP3, TP4, TP5, TP6, TP7, TP8, TP9, U2, U3: LCSC (none) -> DNP
- D1, D2, D3: LCSC (none) -> C191023
- D4, D5, D6, D7, D8: LCSC (none) -> C2290
- L1: LCSC (none) -> C149588
- Q2, Q3: LCSC (none) -> C105166
- Q4, Q7, Q8: LCSC (none) -> C20917
- Q5: LCSC (none) -> C2149
- R1, R2, R27, R28: LCSC (none) -> C601102
- R10, R29, R30, R32, R38: LCSC (none) -> C11702
- R11, R14, R15, R20, R21, R22, R23, R24, R25, R26, R33, R34, R35, R36, R37, R5, R6, R7, R8, R9: LCSC (none) -> C25744
- R12, R13, R3: LCSC (none) -> C17888
- R18, R19, R31: LCSC (none) -> C25890
- R4: LCSC (none) -> C25756
- U1: LCSC (none) -> C74192
- U4: LCSC (none) -> C141380
- U5: LCSC (none) -> C132291
